File: CPU_Power.kicad_sch (KiCad schematic)
At the start: 0 parts

Commit message: initial commit
Parts:
- added C1: C, symbol Device:C
- added R1: R, symbol Device:R
- added U1, U2: rv1126/rv1109, symbol CPU_Rockchip:rv1126_rv1109
Connections:
- new net: C1.1, R1.1, U1.H14 (VCCIO_VDD_1V8)
- new net GND: C1.2, U2.A1 (VSS_1), U2.A21 (AVSS_1), U2.AA1 (VSS_95), U2.AA10 (VSS_96), U2.AA21 (VSS_97), U2.B12 (VSS_2), U2.C10 (VSS_6), U2.C12 (VSS_7), U2.C3 (VSS_3), U2.C5 (VSS_4), U2.C7 (VSS_5), U2.D12 (VSS_9), U2.D18 (AVSS_2), U2.D9 (VSS_8), U2.E10 (VSS_14), U2.E11 (VSS_15), U2.E12 (VSS_16), U2.E4 (VSS_10), U2.E6 (VSS_11), U2.E8 (VSS_12), U2.E9 (VSS_13), U2.F10 (VSS_22), U2.F11 (VSS_23), U2.F12 (VSS_24), U2.F13 (VSS_25), U2.F14 (AVSS_3), U2.F15 (AVSS_4), U2.F3 (VSS_17), U2.F5 (VSS_18), U2.F7 (VSS_19), U2.F8 (VSS_20), U2.F9 (VSS_21), U2.G10 (VSS_29), U2.G11 (VSS_30), U2.G12 (VSS_31), U2.G13 (VSS_32), U2.G16 (AVSS_5), U2.G17 (AVSS_6), U2.G2 (VSS_26), U2.G5 (VSS_27), U2.G6 (VSS_28), U2.H10 (VSS_37), U2.H15 (VSS_38), U2.H4 (VSS_33), U2.H5 (VSS_34), U2.H6 (VSS_35), U2.H7 (VSS_36), U2.J12 (VSS_41), U2.J14 (VSS_42), U2.J16 (VSS_43), U2.J5 (VSS_39), U2.J6 (VSS_40), U2.K12 (VSS_48), U2.K13 (VSS_49), U2.K14 (VSS_50), U2.K5 (VSS_44), U2.K6 (VSS_45), U2.K8 (VSS_46), U2.K9 (VSS_47), U2.L11 (VSS_54), U2.L12 (VSS_55), U2.L13 (VSS_56), U2.L14 (VSS_57), U2.L16 (VSS_58), U2.L2 (VSS_51), U2.L5 (VSS_52), U2.L6 (VSS_53), U2.M10 (VSS_63), U2.M12 (VSS_64), U2.M13 (VSS_65), U2.M14 (VSS_66), U2.M16 (VSS_67), U2.M3 (VSS_59), U2.M5 (VSS_60), U2.M7 (VSS_61), U2.M8 (VSS_62), U2.N10 (VSS_71), U2.N11 (VSS_72), U2.N13 (VSS_73), U2.N14 (VSS_74), U2.N16 (VSS_75), U2.N5 (VSS_68), U2.N6 (VSS_69), U2.N7 (VSS_70), U2.P14 (VSS_80), U2.P16 (VSS_81), U2.P5 (VSS_76), U2.P7 (VSS_77), U2.P8 (VSS_78), U2.P9 (VSS_79), U2.R1 (VSS_82), U2.R12 (VSS_84), U2.R13 (VSS_85), U2.R14 (VSS_86), U2.R5 (VSS_83), U2.T10 (VSS_89), U2.T14 (VSS_90), U2.T17 (VSS_91), U2.T6 (VSS_87), U2.T9 (VSS_88), U2.V17 (VSS_92), U2.W14 (VSS_94), U2.W9 (VSS_93)
- new net VDD_1V8: R1.2
- new net VDD_ARM: U1.N12 (ARM_VDD_1), U1.P12 (ARM_VDD_2), U1.P13 (ARM_VDD_3)
- new net VDD_LOGIC: U1.H13 (LOGIC_VDD_2), U1.H9 (LOGIC_VDD_1), U1.J13 (LOGIC_VDD_4), U1.J9 (LOGIC_VDD_3), U1.L10 (LOGIC_VDD_5), U1.M11 (LOGIC_VDD_6)
- new net VDD_NPU: U1.H11 (NPU_VDD_1), U1.H12 (NPU_VDD_2), U1.J10 (NPU_VDD_3), U1.J11 (NPU_VDD_4), U1.K10 (NPU_VDD_5), U1.K11 (NPU_VDD_6)
- new net VDD_VEPU: U1.L9 (VEPU_VDD_1), U1.M9 (VEPU_VDD_2), U1.N8 (VEPU_VDD_3), U1.N9 (VEPU_VDD_4)
Other:
- company: (none) -> Qingdao IotPi Information Technology
- title: (none) -> Leaf RV1126 Power
