File: PMIC.kicad_sch (KiCad schematic)
At the start: 0 parts

Commit message: initial commit
Other:
- company: (none) -> Qingdao IotPi Information Technology
- title: (none) -> Leaf RV1126 Power
Changed lines of the file:
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@@
 (kicad_sch (version 20230121) (generator eeschema)
   (paper "A4")
+  (title_block
+    (title "Leaf RV1126 Power")
+    (date "2023-02-23")
+    (rev "1")
+    (company "Qingdao IotPi Information Technology")
+  )
 )

Commit message: PMIC management
Other:
- added sheet PMIC Codec (PMIC_codec.kicad_sch)
- added sheet PMIC DCDC (PMIC_dcdc.kicad_sch)
- added sheet PMIC LDO (PMIC_LDO.kicad_sch)
- added sheet PMIC Management (PMIC_management.kicad_sch)
Changed lines of the file:
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@@
     (company "Qingdao IotPi Information Technology")
   )
+  (sheet (at 115.57 43.18) (size 38.1 29.21) (fields_autoplaced)
+    (stroke (width 0.1524) (type solid))
+    (fill (color 0 0 0 0.0000))
+    (property "Sheetname" "PMIC DCDC" (at 115.57 42.4684 0)
+      (effects (font (size 1.27 1.27)) (justify left bottom))
+    )
+    (property "Sheetfile" "PMIC_dcdc.kicad_sch" (at 115.57 72.9746 0)
+      (effects (font (size 1.27 1.27)) (justify left top))
+    )
+    (instances
+      (project "leaf"
+        (path "/e3b58043-16a3-43c8-9fad-9c9784eebfa4/cc9fb3ac-19c3-47a8-ba7d-678b4d514ff0/46e9a7bf-8506-4399-90d8-57d007223126" (page "14"))
+      )
+    )
+  )
+  (sheet (at 48.26 97.79) (size 39.37 26.67) (fields_autoplaced)
+    (stroke (width 0.1524) (type solid))
+    (fill (color 0 0 0 0.0000))
+    (property "Sheetname" "PMIC LDO" (at 48.26 97.0784 0)
+      (effects (font (size 1.27 1.27)) (justify left bottom))
+    )
+    (property "Sheetfile" "PMIC_LDO.kicad_sch" (at 48.26 125.0446 0)
+      (effects (font (size 1.27 1.27)) (justify left top))
+    )
+    (instances
+      (project "leaf"
+        (path "/e3b58043-16a3-43c8-9fad-9c9784eebfa4/cc9fb3ac-19c3-47a8-ba7d-678b4d514ff0/46e9a7bf-8506-4399-90d8-57d007223126" (page "15"))
+      )
+    )
+  )
+  (sheet (at 48.26 44.45) (size 39.37 27.94) (fields_autoplaced)
+    (stroke (width 0.1524) (type solid))
+    (fill (color 0 0 0 0.0000))
+    (property "Sheetname" "PMIC Management" (at 48.26 43.7384 0)
+      (effects (font (size 1.27 1.27)) (justify left bottom))
+    )
+    (property "Sheetfile" "PMIC_management.kicad_sch" (at 48.26 72.9746 0)
+      (effects (font (size 1.27 1.27)) (justify left top))
+    )
+    (instances
+      (project "leaf"
+        (path "/e3b58043-16a3-43c8-9fad-9c9784eebfa4/cc9fb3ac-19c3-47a8-ba7d-678b4d514ff0/46e9a7bf-8506-4399-90d8-57d007223126" (page "13"))
+      )
+    )
+  )
+  (sheet (at 119.38 97.79) (size 38.1 26.67) (fields_autoplaced)
+    (stroke (width 0.1524) (type solid))
+    (fill (color 0 0 0 0.0000))
+    (property "Sheetname" "PMIC Codec" (at 119.38 97.0784 0)
+      (effects (font (size 1.27 1.27)) (justify left bottom))
+    )
+    (property "Sheetfile" "PMIC_codec.kicad_sch" (at 119.38 125.0446 0)
+      (effects (font (size 1.27 1.27)) (justify left top))
+    )
+    (instances
+      (project "leaf"
+        (path "/e3b58043-16a3-43c8-9fad-9c9784eebfa4/cc9fb3ac-19c3-47a8-ba7d-678b4d514ff0/46e9a7bf-8506-4399-90d8-57d007223126" (page "16"))
+      )
+    )
+  )
 )

Commit message: PMIC DCDC
Other:
- sheet PMIC Management ports: added PMIC_CLK_32K, PMIC_I2C_SCL, PMIC_I2C_SDA, PMIC_INT, PMIC_RESET, PMIC_SLEEP; removed none
- title: Leaf RV1126 Power -> Leaf RV1126 PMIC RK809
Changed lines of the file:
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@@
   (paper "A4")
   (title_block
-    (title "Leaf RV1126 Power")
+    (title "Leaf RV1126 PMIC RK809")
     (date "2023-02-23")
     (rev "1")
@@
       (effects (font (size 1.27 1.27)) (justify left top))
     )
+    (pin "PMIC_I2C_SCL" input (at 48.26 52.07 180)
+      (effects (font (size 1.27 1.27)) (justify left))
+    )
+    (pin "PMIC_CLK_32K" output (at 48.26 55.88 180)
+      (effects (font (size 1.27 1.27)) (justify left))
+    )
+    (pin "PMIC_INT" output (at 48.26 59.69 180)
+      (effects (font (size 1.27 1.27)) (justify left))
+    )
+    (pin "PMIC_SLEEP" input (at 48.26 63.5 180)
+      (effects (font (size 1.27 1.27)) (justify left))
+    )
+    (pin "PMIC_I2C_SDA" bidirectional (at 48.26 67.31 180)
+      (effects (font (size 1.27 1.27)) (justify left))
+    )
+    (pin "PMIC_RESET" bidirectional (at 48.26 48.26 180)
+      (effects (font (size 1.27 1.27)) (justify left))
+    )
     (instances

Commit message: updated: PMIC codec
Other:
- title: Leaf RV1126 PMIC RK809 -> Leaf RV1126 PMIC RK809 Codec
Changed lines of the file:
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@@
   (paper "A4")
   (title_block
-    (title "Leaf RV1126 PMIC RK809")
-    (date "2023-02-23")
+    (title "Leaf RV1126 PMIC RK809 Codec")
+    (date "2023-02-25")
     (rev "1")
     (company "Qingdao IotPi Information Technology")

Commit message: updated: PMIC
Other:
- sheet PMIC Codec ports: added HPL_OUT, HPR_OUT, HP_SNS, I2S_LRCLK_TX, I2S_MCLK, I2S_SCLK_TX, I2S_SDI0, I2S_SDO0, SPKN_OUT, SPKP_OUT; removed none
- sheet PMIC Management ports: added CLK_32K, I2C_SCL, I2C_SDA, INT, RESET, SLEEP; removed PMIC_CLK_32K, PMIC_I2C_SCL, PMIC_I2C_SDA, PMIC_INT, PMIC_RESET, PMIC_SLEEP
Changed lines of the file:
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@@
       (effects (font (size 1.27 1.27)) (justify left top))
     )
-    (pin "PMIC_I2C_SCL" input (at 48.26 52.07 180)
+    (pin "I2C_SDA" bidirectional (at 48.26 50.8 180)
       (effects (font (size 1.27 1.27)) (justify left))
     )
-    (pin "PMIC_CLK_32K" output (at 48.26 55.88 180)
+    (pin "CLK_32K" output (at 48.26 55.88 180)
       (effects (font (size 1.27 1.27)) (justify left))
     )
-    (pin "PMIC_INT" output (at 48.26 59.69 180)
+    (pin "INT" output (at 48.26 59.69 180)
       (effects (font (size 1.27 1.27)) (justify left))
     )
-    (pin "PMIC_SLEEP" input (at 48.26 63.5 180)
+    (pin "I2C_SCL" input (at 48.26 46.99 180)
       (effects (font (size 1.27 1.27)) (justify left))
     )
-    (pin "PMIC_I2C_SDA" bidirectional (at 48.26 67.31 180)
+    (pin "SLEEP" input (at 48.26 63.5 180)
       (effects (font (size 1.27 1.27)) (justify left))
     )
-    (pin "PMIC_RESET" bidirectional (at 48.26 48.26 180)
+    (pin "RESET" bidirectional (at 48.26 67.31 180)
       (effects (font (size 1.27 1.27)) (justify left))
     )
@@
       (effects (font (size 1.27 1.27)) (justify left top))
     )
+    (pin "SPKN_OUT" input (at 157.48 109.22 0)
+      (effects (font (size 1.27 1.27)) (justify right))
+    )
+    (pin "HP_SNS" input (at 157.48 111.76 0)
+      (effects (font (size 1.27 1.27)) (justify right))
+    )
+    (pin "HPR_OUT" input (at 157.48 114.3 0)
+      (effects (font (size 1.27 1.27)) (justify right))
+    )
+    (pin "HPL_OUT" input (at 157.48 116.84 0)
+      (effects (font (size 1.27 1.27)) (justify right))
+    )
+    (pin "I2S_SDI0" input (at 119.38 106.68 180)
+      (effects (font (size 1.27 1.27)) (justify left))
+    )
+    (pin "SPKP_OUT" input (at 157.48 106.68 0)
+      (effects (font (size 1.27 1.27)) (justify right))
+    )
+    (pin "I2S_MCLK" input (at 119.38 109.22 180)
+      (effects (font (size 1.27 1.27)) (justify left))
+    )
+    (pin "I2S_LRCLK_TX" input (at 119.38 111.76 180)
+      (effects (font (size 1.27 1.27)) (justify left))
+    )
+    (pin "I2S_SCLK_TX" input (at 119.38 114.3 180)
+      (effects (font (size 1.27 1.27)) (justify left))
+    )
+    (pin "I2S_SDO0" input (at 119.38 116.84 180)
+      (effects (font (size 1.27 1.27)) (justify left))
+    )
     (instances

Commit message: updated: titles
Other:
- sheet PMIC Codec renamed RK809 Codec
- sheet PMIC DCDC renamed RK809 DCDC
- sheet PMIC LDO renamed RK809 LDO
- sheet PMIC Management renamed RK809 Management
- title: Leaf RV1126 PMIC RK809 Codec -> Leaf RV1126 PMIC
Changed lines of the file:
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@@
   (paper "A4")
   (title_block
-    (title "Leaf RV1126 PMIC RK809 Codec")
+    (title "Leaf RV1126 PMIC")
     (date "2023-02-25")
     (rev "1")
@@
     (stroke (width 0.1524) (type solid))
     (fill (color 0 0 0 0.0000))
-    (property "Sheetname" "PMIC DCDC" (at 115.57 42.4684 0)
+    (property "Sheetname" "RK809 DCDC" (at 115.57 42.4684 0)
       (effects (font (size 1.27 1.27)) (justify left bottom))
     )
@@
     (stroke (width 0.1524) (type solid))
     (fill (color 0 0 0 0.0000))
-    (property "Sheetname" "PMIC LDO" (at 48.26 97.0784 0)
+    (property "Sheetname" "RK809 LDO" (at 48.26 97.0784 0)
       (effects (font (size 1.27 1.27)) (justify left bottom))
     )
@@
     (stroke (width 0.1524) (type solid))
     (fill (color 0 0 0 0.0000))
-    (property "Sheetname" "PMIC Management" (at 48.26 43.7384 0)
+    (property "Sheetname" "RK809 Management" (at 48.26 43.7384 0)
       (effects (font (size 1.27 1.27)) (justify left bottom))
     )
@@
     (stroke (width 0.1524) (type solid))
     (fill (color 0 0 0 0.0000))
-    (property "Sheetname" "PMIC Codec" (at 119.38 97.0784 0)
+    (property "Sheetname" "RK809 Codec" (at 119.38 97.0784 0)
       (effects (font (size 1.27 1.27)) (justify left bottom))
     )
