File: SDCard.kicad_sch (KiCad schematic)
At the start: 0 parts

Commit message: PMIC DCDC
Other:
- title: Leaf RV1126 Power -> Leaf RV1126 PMIC RK809
Changed lines of the file:
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@@
   (paper "A4")
   (title_block
-    (title "Leaf RV1126 Power")
+    (title "Leaf RV1126 PMIC RK809")
     (date "2023-02-23")
     (rev "1")

Commit message: updated: PMIC codec
Other:
- title: Leaf RV1126 PMIC RK809 -> Leaf RV1126 PMIC RK809 Codec
Changed lines of the file:
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@@
   (paper "A4")
   (title_block
-    (title "Leaf RV1126 PMIC RK809")
-    (date "2023-02-23")
+    (title "Leaf RV1126 PMIC RK809 Codec")
+    (date "2023-02-25")
     (rev "1")
     (company "Qingdao IotPi Information Technology")

Commit message: updated: titles
Other:
- title: Leaf RV1126 PMIC RK809 Codec -> Leaf RV1126 RK809 SDCard
Changed lines of the file:
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@@
   (paper "A4")
   (title_block
-    (title "Leaf RV1126 PMIC RK809 Codec")
+    (title "Leaf RV1126 RK809 SDCard")
     (date "2023-02-25")
     (rev "1")
