File: SDCard.kicad_sch (KiCad schematic)
At the start: 19 parts, among them J1 Micro_SD_Card_Det1, U1 rv1126/rv1109

Commit message: updated PMIC
Parts:
- J1: footprint Connector_Card:microSD_HC_Wuerth_693072010801 -> Leaf_Connector:microSD; LCSC (none) -> C2982548; Model (none) -> TF-123-ARP9H17; Vendor (none) -> XUNPU(讯普)
Changed lines of the file:
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@@
       (effects (font (size 1.27 1.27)))
     )
-    (property "Footprint" "Connector_Card:microSD_HC_Wuerth_693072010801" (at 0 99.06 0)
+    (property "Footprint" "Leaf_Connector:microSD" (at 0 99.06 0)
       (effects (font (size 1.27 1.27)) hide)
     )
-    (property "Datasheet" "https://datasheet.lcsc.com/lcsc/2110151630_XKB-Connectivity-XKTF-015-N_C381082.pdf" (at 52.07 114.3 0)
+    (property "Datasheet" "" (at 52.07 114.3 0)
       (effects (font (size 1.27 1.27)) hide)
     )
+    (property "Description" "MicroSD卡(TF卡),卡连接方式:拔插式,工作温度范围:-25℃~+85℃,本体最大高度:1.7mm,焊接温度(最大值):260℃,触头材质:C5191,触头镀层:金,连接器类型:卡座" (at 52.07 116.84 0)
+      (effects (font (size 1.27 1.27)) hide)
+    )
+    (property "LCSC" "C2982548" (at 52.07 116.84 0)
+      (effects (font (size 1.27 1.27)) hide)
+    )
+    (property "Model" "TF-123-ARP9H17" (at 52.07 116.84 0)
+      (effects (font (size 1.27 1.27)) hide)
+    )
+    (property "Vendor" "XUNPU(讯普)" (at 52.07 116.84 0)
+      (effects (font (size 1.27 1.27)) hide)
+    )
