File: DDR_resistors.kicad_sch (KiCad schematic)
At the start: 9 parts

Commit message: updated DDR
Parts:
- added C79: 100pF C0G 50V, Capacitor_SMD:C_0402_1005Metric, symbol Device:C
- added R26 (x2): 0R 1%, Resistor_SMD:R_0402_1005Metric, symbol Device:R
- added R26 (x3): 49.9R 1%, Resistor_SMD:R_0402_1005Metric, symbol Device:R
Connections:
- new net: C79.1, R26.2, R26.2
- new net DDR_CLKN: R26.2
- new net DDR_CLKP: R26.2
- new net DDR_RASn: R26.2
- new net GND: C79.2
- new net SoC_CLKN: R26.1, R26.1
- new net SoC_CLKP: R26.1, R26.1
- new net SoC_RASn: R26.1
Other:
- note added: "DNP"
