File: Ethernet.kicad_sch (KiCad schematic)
At the start: 0 parts

Commit message: Updated:
Added Display
Rename DDR to DDR3
Parts:
- added U1: rv1126/rv1109, symbol CPU_Rockchip:rv1126_rv1109

Commit message: updated footprints
Parts:
- U1: footprint (none) -> Rockchip_SoC:Rockchip_RV1126_FCCSP409LD_14.0x14.0mm
Changed lines of the file:
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@@
       (effects (font (size 1.27 1.27)))
     )
-    (property "Footprint" "" (at 254 116.84 0)
+    (property "Footprint" "Rockchip_SoC:Rockchip_RV1126_FCCSP409LD_14.0x14.0mm" (at 254 116.84 0)
       (effects (font (size 1.27 1.27)) hide)
     )
@@
       (effects (font (size 1.27 1.27)))
     )
-    (property "Footprint" "" (at 115.57 83.82 0)
+    (property "Footprint" "Rockchip_SoC:Rockchip_RV1126_FCCSP409LD_14.0x14.0mm" (at 115.57 83.82 0)
       (effects (font (size 1.27 1.27)) hide)
     )
