File: eMMC.kicad_sch (KiCad schematic)
At the start: 18 parts, among them U1 rv1126/rv1109, U5 MTFC4GACAJCN

Commit message: updated footprints
Parts:
- U1: footprint (none) -> Rockchip_SoC:Rockchip_RV1126_FCCSP409LD_14.0x14.0mm
- U3: renamed from U5; footprint (none) -> Memory_micron:Micron_eMMC_FBGA-153_11.5x13.0mm
- renumbered TP2 to TP1
Changed lines of the file:
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@@
         )
         (path "/e3b58043-16a3-43c8-9fad-9c9784eebfa4/0d403b82-6ed8-44f7-a148-d104315eeb81"
-          (reference "R52") (unit 1)
+          (reference "R14") (unit 1)
         )
       )
@@
   (symbol (lib_id "power:GND") (at 223.52 102.87 0) (unit 1)
     (in_bom yes) (on_board yes) (dnp no)
-    (property "Reference" "#PWR093" (at 223.52 109.22 0)
+    (property "Reference" "#PWR015" (at 223.52 109.22 0)
       (effects (font (size 1.27 1.27)) hide)
     )
@@
       (project "leaf"
         (path "/e3b58043-16a3-43c8-9fad-9c9784eebfa4/0d403b82-6ed8-44f7-a148-d104315eeb81"
-          (reference "#PWR093") (unit 1)
+          (reference "#PWR015") (unit 1)
         )
       )
@@
         )
         (path "/e3b58043-16a3-43c8-9fad-9c9784eebfa4/0d403b82-6ed8-44f7-a148-d104315eeb81"
-          (reference "C112") (unit 1)
+          (reference "C8") (unit 1)
         )
       )
@@
   (symbol (lib_id "power:GND") (at 245.11 133.35 0) (unit 1)
     (in_bom yes) (on_board yes) (dnp no) (fields_autoplaced)
-    (property "Reference" "#PWR091" (at 245.11 139.7 0)
+    (property "Reference" "#PWR018" (at 245.11 139.7 0)
       (effects (font (size 1.27 1.27)) hide)
     )
@@
       (project "leaf"
         (path "/e3b58043-16a3-43c8-9fad-9c9784eebfa4/0d403b82-6ed8-44f7-a148-d104315eeb81"
-          (reference "#PWR091") (unit 1)
+          (reference "#PWR018") (unit 1)
         )
       )
@@
   (symbol (lib_id "Connector:TestPoint_2Pole") (at 190.5 151.13 90) (unit 1)
     (in_bom yes) (on_board yes) (dnp no) (fields_autoplaced)
-    (property "Reference" "TP2" (at 191.897 150.4863 90)
+    (property "Reference" "TP1" (at 191.897 150.4863 90)
       (effects (font (size 1.27 1.27)) (justify right))
     )
@@
       (project "leaf"
         (path "/e3b58043-16a3-43c8-9fad-9c9784eebfa4/0d403b82-6ed8-44f7-a148-d104315eeb81"
-          (reference "TP2") (unit 1)
+          (reference "TP1") (unit 1)
         )
       )
@@
         )
         (path "/e3b58043-16a3-43c8-9fad-9c9784eebfa4/0d403b82-6ed8-44f7-a148-d104315eeb81"
-          (reference "R54") (unit 1)
+          (reference "R17") (unit 1)
         )
       )
@@
         )
         (path "/e3b58043-16a3-43c8-9fad-9c9784eebfa4/0d403b82-6ed8-44f7-a148-d104315eeb81"
-          (reference "R50") (unit 1)
+          (reference "R12") (unit 1)
         )
       )
@@
   (symbol (lib_id "Memory_eMMC:MTFC4GACAJCN") (at 38.1 171.45 0) (unit 2)
     (in_bom yes) (on_board yes) (dnp no)
-    (property "Reference" "U5" (at 17.78 149.86 0)
+    (property "Reference" "U3" (at 17.78 149.86 0)
       (effects (font (size 1.27 1.27)) (justify left))
     )
@@
       (effects (font (size 1.27 1.27)) (justify left))
     )
-    (property "Footprint" "" (at 29.21 166.37 0)
+    (property "Footprint" "Memory_micron:Micron_eMMC_FBGA-153_11.5x13.0mm" (at 29.21 166.37 0)
       (effects (font (size 1.27 1.27)) hide)
     )
@@
       (project "leaf"
         (path "/e3b58043-16a3-43c8-9fad-9c9784eebfa4/0d403b82-6ed8-44f7-a148-d104315eeb81"
-          (reference "U5") (unit 2)
+          (reference "U3") (unit 2)
         )
       )
@@
   (symbol (lib_id "power:GND") (at 190.5 157.48 0) (unit 1)
     (in_bom yes) (on_board yes) (dnp no) (fields_autoplaced)
-    (property "Reference" "#PWR095" (at 190.5 163.83 0)
+    (property "Reference" "#PWR013" (at 190.5 163.83 0)
       (effects (font (size 1.27 1.27)) hide)
     )
@@
       (project "leaf"
         (path "/e3b58043-16a3-43c8-9fad-9c9784eebfa4/0d403b82-6ed8-44f7-a148-d104315eeb81"
-          (reference "#PWR095") (unit 1)
+          (reference "#PWR013") (unit 1)
         )
       )
@@
   (symbol (lib_id "power:GND") (at 245.11 88.9 0) (unit 1)
     (in_bom yes) (on_board yes) (dnp no) (fields_autoplaced)
-    (property "Reference" "#PWR090" (at 245.11 95.25 0)
+    (property "Reference" "#PWR017" (at 245.11 95.25 0)
       (effects (font (size 1.27 1.27)) hide)
     )
@@
       (project "leaf"
         (path "/e3b58043-16a3-43c8-9fad-9c9784eebfa4/0d403b82-6ed8-44f7-a148-d104315eeb81"
-          (reference "#PWR090") (unit 1)
+          (reference "#PWR017") (unit 1)
         )
       )
@@
         )
         (path "/e3b58043-16a3-43c8-9fad-9c9784eebfa4/0d403b82-6ed8-44f7-a148-d104315eeb81"
-          (reference "R51") (unit 1)
+          (reference "R13") (unit 1)
         )
       )
@@
   (symbol (lib_id "power:GND") (at 99.06 191.77 0) (unit 1)
     (in_bom yes) (on_board yes) (dnp no) (fields_autoplaced)
-    (property "Reference" "#PWR089" (at 99.06 198.12 0)
+    (property "Reference" "#PWR012" (at 99.06 198.12 0)
       (effects (font (size 1.27 1.27)) hide)
     )
@@
       (project "leaf"
         (path "/e3b58043-16a3-43c8-9fad-9c9784eebfa4/0d403b82-6ed8-44f7-a148-d104315eeb81"
-          (reference "#PWR089") (unit 1)
+          (reference "#PWR012") (unit 1)
         )
       )
@@
         )
         (path "/e3b58043-16a3-43c8-9fad-9c9784eebfa4/0d403b82-6ed8-44f7-a148-d104315eeb81"
-          (reference "R55") (unit 1)
+          (reference "R16") (unit 1)
         )
       )
@@
   (symbol (lib_name "MTFC4GACAJCN_1") (lib_id "Memory_eMMC:MTFC4GACAJCN") (at 187.96 53.34 0) (unit 1)
     (in_bom yes) (on_board yes) (dnp no) (fields_autoplaced)
-    (property "Reference" "U5" (at 187.96 31.4071 0)
+    (property "Reference" "U3" (at 187.96 31.4071 0)
       (effects (font (size 1.27 1.27)))
     )
@@
       (effects (font (size 1.27 1.27)))
     )
-    (property "Footprint" "" (at 179.07 48.26 0)
+    (property "Footprint" "Memory_micron:Micron_eMMC_FBGA-153_11.5x13.0mm" (at 179.07 48.26 0)
       (effects (font (size 1.27 1.27)) hide)
     )
@@
       (project "leaf"
         (path "/e3b58043-16a3-43c8-9fad-9c9784eebfa4/0d403b82-6ed8-44f7-a148-d104315eeb81"
-          (reference "U5") (unit 1)
+          (reference "U3") (unit 1)
         )
       )
@@
         )
         (path "/e3b58043-16a3-43c8-9fad-9c9784eebfa4/0d403b82-6ed8-44f7-a148-d104315eeb81"
-          (reference "C113") (unit 1)
+          (reference "C10") (unit 1)
         )
       )
@@
   (symbol (lib_id "power:GND") (at 223.52 80.01 0) (unit 1)
     (in_bom yes) (on_board yes) (dnp no) (fields_autoplaced)
-    (property "Reference" "#PWR094" (at 223.52 86.36 0)
+    (property "Reference" "#PWR014" (at 223.52 86.36 0)
       (effects (font (size 1.27 1.27)) hide)
     )
@@
       (project "leaf"
         (path "/e3b58043-16a3-43c8-9fad-9c9784eebfa4/0d403b82-6ed8-44f7-a148-d104315eeb81"
-          (reference "#PWR094") (unit 1)
+          (reference "#PWR014") (unit 1)
         )
       )
@@
         )
         (path "/e3b58043-16a3-43c8-9fad-9c9784eebfa4/0d403b82-6ed8-44f7-a148-d104315eeb81"
-          (reference "R53") (unit 1)
+          (reference "R15") (unit 1)
         )
       )
@@
         )
         (path "/e3b58043-16a3-43c8-9fad-9c9784eebfa4/0d403b82-6ed8-44f7-a148-d104315eeb81"
-          (reference "R57") (unit 1)
+          (reference "R19") (unit 1)
         )
       )
@@
         )
         (path "/e3b58043-16a3-43c8-9fad-9c9784eebfa4/0d403b82-6ed8-44f7-a148-d104315eeb81"
-          (reference "C114") (unit 1)
+          (reference "C12") (unit 1)
         )
       )
@@
         )
         (path "/e3b58043-16a3-43c8-9fad-9c9784eebfa4/0d403b82-6ed8-44f7-a148-d104315eeb81"
-          (reference "C111") (unit 1)
+          (reference "C6") (unit 1)
         )
       )
@@
         )
         (path "/e3b58043-16a3-43c8-9fad-9c9784eebfa4/0d403b82-6ed8-44f7-a148-d104315eeb81"
-          (reference "R56") (unit 1)
+          (reference "R18") (unit 1)
         )
       )
@@
       (effects (font (size 1.27 1.27)))
     )
-    (property "Footprint" "" (at 100.33 86.36 0)
+    (property "Footprint" "Rockchip_SoC:Rockchip_RV1126_FCCSP409LD_14.0x14.0mm" (at 100.33 86.36 0)
       (effects (font (size 1.27 1.27)) hide)
     )
@@
         )
         (path "/e3b58043-16a3-43c8-9fad-9c9784eebfa4/0d403b82-6ed8-44f7-a148-d104315eeb81"
-          (reference "C115") (unit 1)
+          (reference "C9") (unit 1)
         )
       )
@@
         )
         (path "/e3b58043-16a3-43c8-9fad-9c9784eebfa4/0d403b82-6ed8-44f7-a148-d104315eeb81"
-          (reference "C116") (unit 1)
+          (reference "C11") (unit 1)
         )
       )
@@
   (symbol (lib_id "power:GND") (at 223.52 129.54 0) (unit 1)
     (in_bom yes) (on_board yes) (dnp no) (fields_autoplaced)
-    (property "Reference" "#PWR092" (at 223.52 135.89 0)
+    (property "Reference" "#PWR016" (at 223.52 135.89 0)
       (effects (font (size 1.27 1.27)) hide)
     )
@@
       (project "leaf"
         (path "/e3b58043-16a3-43c8-9fad-9c9784eebfa4/0d403b82-6ed8-44f7-a148-d104315eeb81"
-          (reference "#PWR092") (unit 1)
+          (reference "#PWR016") (unit 1)
         )
       )
@@
   (symbol (lib_id "power:GND") (at 71.12 144.78 0) (unit 1)
     (in_bom yes) (on_board yes) (dnp no) (fields_autoplaced)
-    (property "Reference" "#PWR088" (at 71.12 151.13 0)
+    (property "Reference" "#PWR011" (at 71.12 151.13 0)
       (effects (font (size 1.27 1.27)) hide)
     )
@@
       (project "leaf"
         (path "/e3b58043-16a3-43c8-9fad-9c9784eebfa4/0d403b82-6ed8-44f7-a148-d104315eeb81"
-          (reference "#PWR088") (unit 1)
+          (reference "#PWR011") (unit 1)
         )
       )
@@
         )
         (path "/e3b58043-16a3-43c8-9fad-9c9784eebfa4/0d403b82-6ed8-44f7-a148-d104315eeb81"
-          (reference "C117") (unit 1)
-        )
-      )
+          (reference "C7") (unit 1)
+        )
+      )

Commit message: updated Capacitors
Parts:
- C57: value 4.7Vf X5R 6.3V -> 4.7uF X5R 10V; LCSC (none) -> C77004; Model (none) -> GRM155R61A475KEAAD; Vendor (none) -> muRata(村田)
- C57: LCSC (none) -> C76934; Model (none) -> GRM033R61A104KE15D; Vendor (none) -> muRata(村田)
Changed lines of the file:
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@@
       (effects (font (size 1.27 1.27)) (justify left))
     )
-    (property "Value" "4.7Vf X5R 6.3V" (at 241.3 83.82 90)
+    (property "Value" "4.7uF X5R 10V" (at 241.3 83.82 90)
       (effects (font (size 1.27 1.27)) (justify left))
     )
@@
     )
     (property "Datasheet" "~" (at 245.11 73.66 0)
+      (effects (font (size 1.27 1.27)) hide)
+    )
+    (property "LCSC" "C77004" (at 245.11 73.66 90)
+      (effects (font (size 1.27 1.27)) hide)
+    )
+    (property "Description" "容值: 4.7uF 精度: ±10% 额定电压: 10V 材质(温度系数): X5R 材质:X5R" (at 245.11 73.66 90)
+      (effects (font (size 1.27 1.27)) hide)
+    )
+    (property "Model" "GRM155R61A475KEAAD" (at 245.11 73.66 90)
+      (effects (font (size 1.27 1.27)) hide)
+    )
+    (property "Vendor" "muRata(村田) " (at 245.11 73.66 90)
       (effects (font (size 1.27 1.27)) hide)
     )
@@
     )
     (property "Datasheet" "~" (at 71.12 134.62 0)
+      (effects (font (size 1.27 1.27)) hide)
+    )
+    (property "Description" "容值: 100nF 精度: ±10% 额定电压: 10V 材质(温度系数): X5R 材质:X5R" (at 71.12 134.62 0)
+      (effects (font (size 1.27 1.27)) hide)
+    )
+    (property "LCSC" "C76934" (at 71.12 134.62 0)
+      (effects (font (size 1.27 1.27)) hide)
+    )
+    (property "Model" "GRM033R61A104KE15D" (at 71.12 134.62 0)
+      (effects (font (size 1.27 1.27)) hide)
+    )
+    (property "Vendor" "muRata(村田)" (at 71.12 134.62 0)
       (effects (font (size 1.27 1.27)) hide)
     )
@@
       (effects (font (size 1.27 1.27)) (justify left))
     )
-    (property "Value" "4.7Vf X5R 6.3V" (at 241.3 128.27 90)
+    (property "Value" "4.7uF X5R 10V" (at 241.3 128.27 90)
       (effects (font (size 1.27 1.27)) (justify left))
     )
@@
     )
     (property "Datasheet" "~" (at 245.11 118.11 0)
+      (effects (font (size 1.27 1.27)) hide)
+    )
+    (property "Description" "容值: 4.7uF 精度: ±10% 额定电压: 10V 材质(温度系数): X5R 材质:X5R" (at 245.11 118.11 0)
+      (effects (font (size 1.27 1.27)) hide)
+    )
+    (property "LCSC" "C77004" (at 245.11 118.11 0)
+      (effects (font (size 1.27 1.27)) hide)
+    )
+    (property "Model" "GRM155R61A475KEAAD" (at 245.11 118.11 0)
+      (effects (font (size 1.27 1.27)) hide)
+    )
+    (property "Vendor" "muRata(村田) " (at 245.11 118.11 0)
       (effects (font (size 1.27 1.27)) hide)
     )
@@
       (effects (font (size 1.27 1.27)) (justify left))
     )
-    (property "Value" "4.7Vf X5R 6.3V" (at 219.71 133.35 90)
+    (property "Value" "4.7uF X5R 10V" (at 219.71 133.35 90)
       (effects (font (size 1.27 1.27)) (justify left))
     )
@@
       (effects (font (size 1.27 1.27)) hide)
     )
+    (property "Description" "容值: 4.7uF 精度: ±10% 额定电压: 10V 材质(温度系数): X5R 材质:X5R" (at 223.52 123.19 0)
+      (effects (font (size 1.27 1.27)) hide)
+    )
+    (property "LCSC" "C77004" (at 223.52 123.19 0)
+      (effects (font (size 1.27 1.27)) hide)
+    )
+    (property "Model" "GRM155R61A475KEAAD" (at 223.52 123.19 0)
+      (effects (font (size 1.27 1.27)) hide)
+    )
+    (property "Vendor" "muRata(村田) " (at 223.52 123.19 0)
+      (effects (font (size 1.27 1.27)) hide)
+    )

Commit message: updated LCSC selection of capacitors
Parts:
- C57: value 100nF X5R 16V -> 100nF X5R 6.3V; footprint Capacitor_SMD:C_0402_1005Metric -> Capacitor_SMD:C_0201_0603Metric; LCSC (none) -> C76934; Model (none) -> GRM033R61A104KE15D; Vendor (none) -> muRata(村田)
- R40: now left out of the parts list
Connections:
- net VCCIO_FLASH is gone; now on net VCC_1V8: C57.1, C57.1, C57.1, C57.1, R40.2, R40.2, R40.2, R40.2, U1.P6 (VCCIO1_VDD), U3.C6 (V_{CCQ}), U3.M4 (V_{CCQ}), U3.N4 (V_{CCQ}), U3.P3 (V_{CCQ}), U3.P5 (V_{CCQ})
Changed lines of the file:
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@@
   (junction (at 99.06 170.18) (diameter 0) (color 0 0 0 0)
   )
+  (junction (at 71.12 110.49) (diameter 0) (color 0 0 0 0)
+  )
   (junction (at 223.52 41.91) (diameter 0) (color 0 0 0 0)
   )
@@
   )
   (junction (at 223.52 101.6) (diameter 0) (color 0 0 0 0)
+  )
+  (junction (at 29.21 110.49) (diameter 0) (color 0 0 0 0)
   )
   (junction (at 223.52 54.61) (diameter 0) (color 0 0 0 0)
@@
     (stroke (width 0) (type default))
   )
-  (wire (pts (xy 71.12 105.41) (xy 71.12 114.3))
+  (wire (pts (xy 71.12 105.41) (xy 71.12 110.49))
     (stroke (width 0) (type default))
   )
@@
     (stroke (width 0) (type default))
   )
+  (wire (pts (xy 29.21 110.49) (xy 29.21 114.3))
+    (stroke (width 0) (type default))
+  )
   (wire (pts (xy 212.09 93.98) (xy 223.52 93.98))
     (stroke (width 0) (type default))
@@
     (stroke (width 0) (type default))
   )
+  (wire (pts (xy 71.12 110.49) (xy 71.12 114.3))
+    (stroke (width 0) (type default))
+  )
   (wire (pts (xy 223.52 115.57) (xy 223.52 119.38))
     (stroke (width 0) (type default))
@@
     (stroke (width 0) (type default))
   )
-  (wire (pts (xy 29.21 109.22) (xy 29.21 114.3))
+  (wire (pts (xy 29.21 109.22) (xy 29.21 110.49))
     (stroke (width 0) (type default))
   )
@@
   )
   (wire (pts (xy 223.52 96.52) (xy 223.52 99.06))
+    (stroke (width 0) (type default))
+  )
+  (wire (pts (xy 29.21 110.49) (xy 71.12 110.49))
     (stroke (width 0) (type default))
   )
@@
   )
   (symbol (lib_id "Device:R") (at 50.8 114.3 90) (unit 1)
-    (in_bom yes) (on_board yes) (dnp no)
+    (in_bom no) (on_board no) (dnp no)
     (property "Reference" "R40" (at 55.88 113.03 90)
       (effects (font (size 1.27 1.27)))
@@
   )
   (symbol (lib_id "Device:R") (at 50.8 127 90) (unit 1)
-    (in_bom yes) (on_board yes) (dnp no)
+    (in_bom no) (on_board no) (dnp no)
     (property "Reference" "R40" (at 55.88 125.73 90)
       (effects (font (size 1.27 1.27)))
@@
       (effects (font (size 1.27 1.27)) (justify left))
     )
-    (property "Value" "100nF X5R 16V" (at 251.46 83.82 90)
+    (property "Value" "100nF X5R 6.3V" (at 251.46 83.82 90)
       (effects (font (size 1.27 1.27)) (justify left))
     )
-    (property "Footprint" "Capacitor_SMD:C_0402_1005Metric" (at 256.2352 77.47 0)
+    (property "Footprint" "Capacitor_SMD:C_0201_0603Metric" (at 256.2352 77.47 0)
       (effects (font (size 1.27 1.27)) hide)
     )
     (property "Datasheet" "~" (at 255.27 73.66 0)
+      (effects (font (size 1.27 1.27)) hide)
+    )
+    (property "Description" "容值: 100nF 精度: ±10% 额定电压: 10V 材质(温度系数): X5R 材质:X5R" (at 255.27 73.66 0)
+      (effects (font (size 1.27 1.27)) hide)
+    )
+    (property "Model" "GRM033R61A104KE15D" (at 255.27 73.66 0)
+      (effects (font (size 1.27 1.27)) hide)
+    )
+    (property "Vendor" "muRata(村田)" (at 255.27 73.66 0)
+      (effects (font (size 1.27 1.27)) hide)
+    )
+    (property "LCSC" "C76934" (at 255.27 73.66 0)
       (effects (font (size 1.27 1.27)) hide)
     )
@@
       (effects (font (size 1.27 1.27)) (justify left))
     )
-    (property "Value" "100nF X5R 16V" (at 260.35 83.82 90)
+    (property "Value" "100nF X5R 6.3V" (at 260.35 83.82 90)
       (effects (font (size 1.27 1.27)) (justify left))
     )
-    (property "Footprint" "Capacitor_SMD:C_0402_1005Metric" (at 265.1252 77.47 0)
+    (property "Footprint" "Capacitor_SMD:C_0201_0603Metric" (at 265.1252 77.47 0)
       (effects (font (size 1.27 1.27)) hide)
     )
     (property "Datasheet" "~" (at 264.16 73.66 0)
+      (effects (font (size 1.27 1.27)) hide)
+    )
+    (property "Description" "容值: 100nF 精度: ±10% 额定电压: 10V 材质(温度系数): X5R 材质:X5R" (at 264.16 73.66 0)
+      (effects (font (size 1.27 1.27)) hide)
+    )
+    (property "Model" "GRM033R61A104KE15D" (at 264.16 73.66 0)
+      (effects (font (size 1.27 1.27)) hide)
+    )
+    (property "Vendor" "muRata(村田)" (at 264.16 73.66 0)
+      (effects (font (size 1.27 1.27)) hide)
+    )
+    (property "LCSC" "C76934" (at 264.16 73.66 0)
       (effects (font (size 1.27 1.27)) hide)
     )
@@
       (effects (font (size 1.27 1.27)) (justify left))
     )
-    (property "Value" "100nF X5R 16V" (at 251.46 128.27 90)
+    (property "Value" "100nF X5R 6.3V" (at 251.46 128.27 90)
       (effects (font (size 1.27 1.27)) (justify left))
     )
-    (property "Footprint" "Capacitor_SMD:C_0402_1005Metric" (at 256.2352 121.92 0)
+    (property "Footprint" "Capacitor_SMD:C_0201_0603Metric" (at 256.2352 121.92 0)
       (effects (font (size 1.27 1.27)) hide)
     )
@@
       (effects (font (size 1.27 1.27)) hide)
     )
+    (property "Description" "容值: 100nF 精度: ±10% 额定电压: 10V 材质(温度系数): X5R 材质:X5R" (at 255.27 118.11 0)
+      (effects (font (size 1.27 1.27)) hide)
+    )
+    (property "Model" "GRM033R61A104KE15D" (at 255.27 118.11 0)
+      (effects (font (size 1.27 1.27)) hide)
+    )
+    (property "Vendor" "muRata(村田)" (at 255.27 118.11 0)
+      (effects (font (size 1.27 1.27)) hide)
+    )
+    (property "LCSC" "C76934" (at 255.27 118.11 0)
+      (effects (font (size 1.27 1.27)) hide)
+    )

Commit message: layout SoC Power and DDR capacitors
Parts:
- C57: LCSC C76934 -> C76928; Model GRM033R61A104KE15D -> GRM033R60J104KE19D
Changed lines of the file:
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@@
       (effects (font (size 1.27 1.27)) hide)
     )
-    (property "Description" "容值: 100nF 精度: ±10% 额定电压: 10V 材质(温度系数): X5R 材质:X5R" (at 255.27 73.66 0)
-      (effects (font (size 1.27 1.27)) hide)
-    )
-    (property "Model" "GRM033R61A104KE15D" (at 255.27 73.66 0)
+    (property "Description" "容值: 100nF 精度: ±10% 额定电压: 6.3V 材质(温度系数): X5R 材质:X5R" (at 255.27 73.66 0)
+      (effects (font (size 1.27 1.27)) hide)
+    )
+    (property "Model" "GRM033R60J104KE19D" (at 255.27 73.66 0)
       (effects (font (size 1.27 1.27)) hide)
     )
@@
       (effects (font (size 1.27 1.27)) hide)
     )
-    (property "LCSC" "C76934" (at 255.27 73.66 0)
+    (property "LCSC" "C76928" (at 255.27 73.66 0)
       (effects (font (size 1.27 1.27)) hide)
     )
@@
       (effects (font (size 1.27 1.27)) hide)
     )
-    (property "Description" "容值: 100nF 精度: ±10% 额定电压: 10V 材质(温度系数): X5R 材质:X5R" (at 264.16 73.66 0)
-      (effects (font (size 1.27 1.27)) hide)
-    )
-    (property "Model" "GRM033R61A104KE15D" (at 264.16 73.66 0)
+    (property "Description" "容值: 100nF 精度: ±10% 额定电压: 6.3V 材质(温度系数): X5R 材质:X5R" (at 264.16 73.66 0)
+      (effects (font (size 1.27 1.27)) hide)
+    )
+    (property "Model" "GRM033R60J104KE19D" (at 264.16 73.66 0)
       (effects (font (size 1.27 1.27)) hide)
     )
@@
       (effects (font (size 1.27 1.27)) hide)
     )
-    (property "LCSC" "C76934" (at 264.16 73.66 0)
+    (property "LCSC" "C76928" (at 264.16 73.66 0)
       (effects (font (size 1.27 1.27)) hide)
     )
@@
       (effects (font (size 1.27 1.27)) hide)
     )
-    (property "Description" "容值: 100nF 精度: ±10% 额定电压: 10V 材质(温度系数): X5R 材质:X5R" (at 71.12 134.62 0)
-      (effects (font (size 1.27 1.27)) hide)
-    )
-    (property "LCSC" "C76934" (at 71.12 134.62 0)
-      (effects (font (size 1.27 1.27)) hide)
-    )
-    (property "Model" "GRM033R61A104KE15D" (at 71.12 134.62 0)
+    (property "Description" "容值: 100nF 精度: ±10% 额定电压: 6.3V 材质(温度系数): X5R 材质:X5R" (at 71.12 134.62 0)
+      (effects (font (size 1.27 1.27)) hide)
+    )
+    (property "LCSC" "C76928" (at 71.12 134.62 0)
+      (effects (font (size 1.27 1.27)) hide)
+    )
+    (property "Model" "GRM033R60J104KE19D" (at 71.12 134.62 0)
       (effects (font (size 1.27 1.27)) hide)
     )
@@
       (effects (font (size 1.27 1.27)) hide)
     )
-    (property "Description" "容值: 100nF 精度: ±10% 额定电压: 10V 材质(温度系数): X5R 材质:X5R" (at 255.27 118.11 0)
-      (effects (font (size 1.27 1.27)) hide)
-    )
-    (property "Model" "GRM033R61A104KE15D" (at 255.27 118.11 0)
+    (property "Description" "容值: 100nF 精度: ±10% 额定电压: 6.3V 材质(温度系数): X5R 材质:X5R" (at 255.27 118.11 0)
+      (effects (font (size 1.27 1.27)) hide)
+    )
+    (property "Model" "GRM033R60J104KE19D" (at 255.27 118.11 0)
       (effects (font (size 1.27 1.27)) hide)
     )
@@
       (effects (font (size 1.27 1.27)) hide)
     )
-    (property "LCSC" "C76934" (at 255.27 118.11 0)
-      (effects (font (size 1.27 1.27)) hide)
-    )
+    (property "LCSC" "C76928" (at 255.27 118.11 0)
+      (effects (font (size 1.27 1.27)) hide)
+    )
