File: Camera.kicad_sch (KiCad schematic)
At the start: 14 parts, among them J2 MIPI-CSI, U1 rv1126/rv1109

Commit message: updated LCSC selection of capacitors
Parts:
- C57: footprint Capacitor_SMD:C_0603_1608Metric -> Capacitor_SMD:C_0402_1005Metric; LCSC (none) -> C77000; Model (none) -> GRM155R61A106ME44D; Vendor (none) -> muRata(村田)
- J2: footprint (none) -> Connector_FFC-FPC:Hirose_FH12-30S-0.5SH_1x30-1MP_P0.50mm_Horizontal
Changed lines of the file:
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@@
       (effects (font (size 1.27 1.27)))
     )
-    (property "Footprint" "" (at 275.59 68.58 0)
+    (property "Footprint" "Connector_FFC-FPC:Hirose_FH12-30S-0.5SH_1x30-1MP_P0.50mm_Horizontal" (at 275.59 68.58 0)
       (effects (font (size 1.27 1.27)) hide)
     )
@@
       (effects (font (size 1.27 1.27)) (justify left))
     )
-    (property "Footprint" "Capacitor_SMD:C_0603_1608Metric" (at 253.6952 132.08 0)
+    (property "Footprint" "Capacitor_SMD:C_0402_1005Metric" (at 253.6952 132.08 0)
       (effects (font (size 1.27 1.27)) hide)
     )
     (property "Datasheet" "~" (at 252.73 128.27 0)
+      (effects (font (size 1.27 1.27)) hide)
+    )
+    (property "Description" "容值: 10uF 精度: ±20% 额定电压: 10V 材质(温度系数): X5R 材质:X5R" (at 252.73 128.27 0)
+      (effects (font (size 1.27 1.27)) hide)
+    )
+    (property "LCSC" "C77000" (at 252.73 128.27 0)
+      (effects (font (size 1.27 1.27)) hide)
+    )
+    (property "Model" "GRM155R61A106ME44D" (at 252.73 128.27 0)
+      (effects (font (size 1.27 1.27)) hide)
+    )
+    (property "Vendor" "muRata(村田)" (at 252.73 128.27 0)
       (effects (font (size 1.27 1.27)) hide)
     )
@@
       (effects (font (size 1.27 1.27)) (justify left))
     )
-    (property "Footprint" "Capacitor_SMD:C_0603_1608Metric" (at 229.5652 132.08 0)
+    (property "Footprint" "Capacitor_SMD:C_0402_1005Metric" (at 229.5652 132.08 0)
       (effects (font (size 1.27 1.27)) hide)
     )
@@
       (effects (font (size 1.27 1.27)) hide)
     )
+    (property "Description" "容值: 10uF 精度: ±20% 额定电压: 10V 材质(温度系数): X5R 材质:X5R" (at 228.6 128.27 0)
+      (effects (font (size 1.27 1.27)) hide)
+    )
+    (property "LCSC" "C77000" (at 228.6 128.27 0)
+      (effects (font (size 1.27 1.27)) hide)
+    )
+    (property "Model" "GRM155R61A106ME44D" (at 228.6 128.27 0)
+      (effects (font (size 1.27 1.27)) hide)
+    )
+    (property "Vendor" "muRata(村田)" (at 228.6 128.27 0)
+      (effects (font (size 1.27 1.27)) hide)
+    )

Commit message: updated foorprints
Parts:
- J2: footprint Connector_FFC-FPC:Hirose_FH12-30S-0.5SH_1x30-1MP_P0.50mm_Horizontal -> Connector_FFC-FPC:Hirose_FH12-24S-0.5SH_1x24-1MP_P0.50mm_Horizontal
Changed lines of the file:
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@@
       (effects (font (size 1.27 1.27)))
     )
-    (property "Footprint" "Connector_FFC-FPC:Hirose_FH12-30S-0.5SH_1x30-1MP_P0.50mm_Horizontal" (at 275.59 68.58 0)
+    (property "Footprint" "Connector_FFC-FPC:Hirose_FH12-24S-0.5SH_1x24-1MP_P0.50mm_Horizontal" (at 275.59 68.58 0)
       (effects (font (size 1.27 1.27)) hide)
     )

Commit message: layout SoC Power and DDR capacitors
Parts:
- C57: LCSC C76934 -> C76928; Model GRM033R61A104KE15D -> GRM033R60J104KE19D
Changed lines of the file:
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@@
       (effects (font (size 1.27 1.27)) hide)
     )
-    (property "Description" "容值: 100nF 精度: ±10% 额定电压: 10V 材质(温度系数): X5R 材质:X5R" (at 275.59 128.27 0)
-      (effects (font (size 1.27 1.27)) hide)
-    )
-    (property "LCSC" "C76934" (at 275.59 128.27 0)
-      (effects (font (size 1.27 1.27)) hide)
-    )
-    (property "Model" "GRM033R61A104KE15D" (at 275.59 128.27 0)
+    (property "Description" "容值: 100nF 精度: ±10% 额定电压: 6.3V 材质(温度系数): X5R 材质:X5R" (at 275.59 128.27 0)
+      (effects (font (size 1.27 1.27)) hide)
+    )
+    (property "LCSC" "C76928" (at 275.59 128.27 0)
+      (effects (font (size 1.27 1.27)) hide)
+    )
+    (property "Model" "GRM033R60J104KE19D" (at 275.59 128.27 0)
       (effects (font (size 1.27 1.27)) hide)
     )
@@
       (effects (font (size 1.27 1.27)) hide)
     )
-    (property "Description" "容值: 100nF 精度: ±10% 额定电压: 10V 材质(温度系数): X5R 材质:X5R" (at 96.52 77.47 0)
-      (effects (font (size 1.27 1.27)) hide)
-    )
-    (property "LCSC" "C76934" (at 96.52 77.47 0)
-      (effects (font (size 1.27 1.27)) hide)
-    )
-    (property "Model" "GRM033R61A104KE15D" (at 96.52 77.47 0)
+    (property "Description" "容值: 100nF 精度: ±10% 额定电压: 6.3V 材质(温度系数): X5R 材质:X5R" (at 96.52 77.47 0)
+      (effects (font (size 1.27 1.27)) hide)
+    )
+    (property "LCSC" "C76928" (at 96.52 77.47 0)
+      (effects (font (size 1.27 1.27)) hide)
+    )
+    (property "Model" "GRM033R60J104KE19D" (at 96.52 77.47 0)
       (effects (font (size 1.27 1.27)) hide)
     )
@@
       (effects (font (size 1.27 1.27)) hide)
     )
-    (property "Description" "容值: 100nF 精度: ±10% 额定电压: 10V 材质(温度系数): X5R 材质:X5R" (at 238.76 128.27 0)
-      (effects (font (size 1.27 1.27)) hide)
-    )
-    (property "LCSC" "C76934" (at 238.76 128.27 0)
-      (effects (font (size 1.27 1.27)) hide)
-    )
-    (property "Model" "GRM033R61A104KE15D" (at 238.76 128.27 0)
+    (property "Description" "容值: 100nF 精度: ±10% 额定电压: 6.3V 材质(温度系数): X5R 材质:X5R" (at 238.76 128.27 0)
+      (effects (font (size 1.27 1.27)) hide)
+    )
+    (property "LCSC" "C76928" (at 238.76 128.27 0)
+      (effects (font (size 1.27 1.27)) hide)
+    )
+    (property "Model" "GRM033R60J104KE19D" (at 238.76 128.27 0)
       (effects (font (size 1.27 1.27)) hide)
     )
@@
       (effects (font (size 1.27 1.27)) hide)
     )
-    (property "Description" "容值: 100nF 精度: ±10% 额定电压: 10V 材质(温度系数): X5R 材质:X5R" (at 64.77 177.8 0)
-      (effects (font (size 1.27 1.27)) hide)
-    )
-    (property "LCSC" "C76934" (at 64.77 177.8 0)
-      (effects (font (size 1.27 1.27)) hide)
-    )
-    (property "Model" "GRM033R61A104KE15D" (at 64.77 177.8 0)
+    (property "Description" "容值: 100nF 精度: ±10% 额定电压: 6.3V 材质(温度系数): X5R 材质:X5R" (at 64.77 177.8 0)
+      (effects (font (size 1.27 1.27)) hide)
+    )
+    (property "LCSC" "C76928" (at 64.77 177.8 0)
+      (effects (font (size 1.27 1.27)) hide)
+    )
+    (property "Model" "GRM033R60J104KE19D" (at 64.77 177.8 0)
       (effects (font (size 1.27 1.27)) hide)
     )
@@
       (effects (font (size 1.27 1.27)) hide)
     )
-    (property "Description" "容值: 100nF 精度: ±10% 额定电压: 10V 材质(温度系数): X5R 材质:X5R" (at 109.22 179.07 0)
-      (effects (font (size 1.27 1.27)) hide)
-    )
-    (property "LCSC" "C76934" (at 109.22 179.07 0)
-      (effects (font (size 1.27 1.27)) hide)
-    )
-    (property "Model" "GRM033R61A104KE15D" (at 109.22 179.07 0)
+    (property "Description" "容值: 100nF 精度: ±10% 额定电压: 6.3V 材质(温度系数): X5R 材质:X5R" (at 109.22 179.07 0)
+      (effects (font (size 1.27 1.27)) hide)
+    )
+    (property "LCSC" "C76928" (at 109.22 179.07 0)
+      (effects (font (size 1.27 1.27)) hide)
+    )
+    (property "Model" "GRM033R60J104KE19D" (at 109.22 179.07 0)
       (effects (font (size 1.27 1.27)) hide)
     )
@@
       (effects (font (size 1.27 1.27)) hide)
     )
-    (property "Description" "容值: 100nF 精度: ±10% 额定电压: 10V 材质(温度系数): X5R 材质:X5R" (at 262.89 128.27 0)
-      (effects (font (size 1.27 1.27)) hide)
-    )
-    (property "LCSC" "C76934" (at 262.89 128.27 0)
-      (effects (font (size 1.27 1.27)) hide)
-    )
-    (property "Model" "GRM033R61A104KE15D" (at 262.89 128.27 0)
-      (effects (font (size 1.27 1.27)) hide)
-    )
+    (property "Description" "容值: 100nF 精度: ±10% 额定电压: 6.3V 材质(温度系数): X5R 材质:X5R" (at 262.89 128.27 0)
+      (effects (font (size 1.27 1.27)) hide)
+    )
+    (property "LCSC" "C76928" (at 262.89 128.27 0)
+      (effects (font (size 1.27 1.27)) hide)
+    )
+    (property "Model" "GRM033R60J104KE19D" (at 262.89 128.27 0)
+      (effects (font (size 1.27 1.27)) hide)
+    )

Commit message: updated Resistors
Parts:
- R40: LCSC (none) -> C966701; Model (none) -> CQ02WGJ0222TCE; Vendor (none) -> UNI-ROYAL(厚声)
Changed lines of the file:
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@@
+      (effects (font (size 1.27 1.27)) hide)
+    )
+    (property "Description" "阻值: 2.2kΩ 精度: ±5% 功率: 0.0625W 温度系数: ±100ppm/℃" (at 41.91 116.84 0)
+      (effects (font (size 1.27 1.27)) hide)
+    )
+    (property "LCSC" "C966701" (at 41.91 116.84 0)
+      (effects (font (size 1.27 1.27)) hide)
+    )
+    (property "Model" "CQ02WGJ0222TCE" (at 41.91 116.84 0)
+      (effects (font (size 1.27 1.27)) hide)
+    )
+    (property "Vendor" "UNI-ROYAL(厚声)" (at 41.91 116.84 0)
       (effects (font (size 1.27 1.27)) hide)
     )
@@
       (effects (font (size 1.27 1.27)) hide)
     )
+    (property "Description" "阻值: 2.2kΩ 精度: ±5% 功率: 0.0625W 温度系数: ±100ppm/℃" (at 52.07 116.84 0)
+      (effects (font (size 1.27 1.27)) hide)
+    )
+    (property "LCSC" "C966701" (at 52.07 116.84 0)
+      (effects (font (size 1.27 1.27)) hide)
+    )
+    (property "Model" "CQ02WGJ0222TCE" (at 52.07 116.84 0)
+      (effects (font (size 1.27 1.27)) hide)
+    )
+    (property "Vendor" "UNI-ROYAL(厚声)" (at 52.07 116.84 0)
+      (effects (font (size 1.27 1.27)) hide)
+    )

Commit message: fix some ERCs
Parts:
- renumbered C57 to C?, R40 to R?

Commit message: updated symbols
Parts:
- R? (x2): LCSC (none) -> C17168; Model (none) -> 0402WGF0000TCE; Vendor (none) -> UNI-ROYAL(厚声)
Changed lines of the file:
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@@
+      (effects (font (size 1.27 1.27)) hide)
+    )
+    (property "Description" "电阻类型: 厚膜电阻 阻值: 0Ω 精度: ±1% 功率: 1/16W 温度系数: ±800ppm/℃ 最大工作电压: 50V 工作" (at 97.79 171.45 0)
+      (effects (font (size 1.27 1.27)) hide)
+    )
+    (property "LCSC" "C17168" (at 97.79 171.45 0)
+      (effects (font (size 1.27 1.27)) hide)
+    )
+    (property "Model" "0402WGF0000TCE" (at 97.79 171.45 0)
+      (effects (font (size 1.27 1.27)) hide)
+    )
+    (property "Vendor" "UNI-ROYAL(厚声)" (at 97.79 171.45 0)
       (effects (font (size 1.27 1.27)) hide)
     )
@@
       (effects (font (size 1.27 1.27)) hide)
     )
+    (property "Description" "电阻类型: 厚膜电阻 阻值: 0Ω 精度: ±1% 功率: 1/16W 温度系数: ±800ppm/℃ 最大工作电压: 50V 工作" (at 53.34 170.18 0)
+      (effects (font (size 1.27 1.27)) hide)
+    )
+    (property "LCSC" "C17168" (at 53.34 170.18 0)
+      (effects (font (size 1.27 1.27)) hide)
+    )
+    (property "Model" "0402WGF0000TCE" (at 53.34 170.18 0)
+      (effects (font (size 1.27 1.27)) hide)
+    )
+    (property "Vendor" "UNI-ROYAL(厚声)" (at 53.34 170.18 0)
+      (effects (font (size 1.27 1.27)) hide)
+    )

Commit message: fixing warnings
Connections:
- net GND: no longer C?.2, C?.2, J2.1 (Pin_1), J2.17 (Pin_17), J2.2 (Pin_2), J2.20 (Pin_20), J2.7 (Pin_7), J2.8 (Pin_8)
- new net GNDA: C?.2, C?.2
- new net GNDD: J2.1 (Pin_1), J2.17 (Pin_17), J2.2 (Pin_2), J2.20 (Pin_20), J2.7 (Pin_7), J2.8 (Pin_8)
Changed lines of the file:
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@@
   (junction (at 41.91 105.41) (diameter 0) (color 0 0 0 0)
-  )
-  (junction (at 135.89 181.61) (diameter 0) (color 0 0 0 0)
   )
   (junction (at 252.73 140.97) (diameter 0) (color 0 0 0 0)
@@
     (stroke (width 0) (type default))
   )
-  (wire (pts (xy 135.89 181.61) (xy 148.59 181.61))
-    (stroke (width 0) (type default))
-  )
   (wire (pts (xy 52.07 120.65) (xy 52.07 125.73))
     (stroke (width 0) (type default))
@@
     (stroke (width 0) (type default))
   )
-  (wire (pts (xy 135.89 184.15) (xy 135.89 181.61))
-    (stroke (width 0) (type default))
-  )
   (wire (pts (xy 238.76 119.38) (xy 228.6 119.38))
     (stroke (width 0) (type default))
@@
     (stroke (width 0) (type default))
   )
-  (wire (pts (xy 148.59 181.61) (xy 148.59 184.15))
-    (stroke (width 0) (type default))
-  )
   (wire (pts (xy 241.3 76.2) (xy 270.51 76.2))
     (stroke (width 0) (type default))
@@
     (stroke (width 0) (type default))
   )
-  (wire (pts (xy 123.19 181.61) (xy 123.19 184.15))
-    (stroke (width 0) (type default))
-  )
   (wire (pts (xy 262.89 119.38) (xy 262.89 124.46))
-    (stroke (width 0) (type default))
-  )
-  (wire (pts (xy 135.89 181.61) (xy 123.19 181.61))
     (stroke (width 0) (type default))
   )
@@
     (property "Intersheetrefs" "${INTERSHEET_REFS}" (at 15.6604 22.86 0)
       (effects (font (size 1.27 1.27)) (justify right) hide)
-    )
-  )
-  (symbol (lib_id "power:GNDA") (at 123.19 184.15 0) (unit 1)
-    (in_bom yes) (on_board yes) (dnp no) (fields_autoplaced)
-    (property "Reference" "#PWR020" (at 123.19 190.5 0)
-      (effects (font (size 1.27 1.27)) hide)
-    )
-    (property "Value" "GNDA" (at 123.19 188.2855 0)
-      (effects (font (size 1.27 1.27)))
-    )
-    (property "Footprint" "" (at 123.19 184.15 0)
-      (effects (font (size 1.27 1.27)) hide)
-    )
-    (property "Datasheet" "" (at 123.19 184.15 0)
-      (effects (font (size 1.27 1.27)) hide)
-    )
-    (pin "1")
-    (instances
-      (project "leaf"
-        (path "/e3b58043-16a3-43c8-9fad-9c9784eebfa4/bca9f05a-f031-46a4-95a9-25be55b42bf6"
-          (reference "#PWR020") (unit 1)
-        )
-      )
     )
   )
@@
     )
   )
-  (symbol (lib_id "power:GND") (at 148.59 184.15 0) (unit 1)
-    (in_bom yes) (on_board yes) (dnp no) (fields_autoplaced)
-    (property "Reference" "#PWR022" (at 148.59 190.5 0)
-      (effects (font (size 1.27 1.27)) hide)
-    )
-    (property "Value" "GND" (at 148.59 188.2855 0)
-      (effects (font (size 1.27 1.27)))
-    )
-    (property "Footprint" "" (at 148.59 184.15 0)
-      (effects (font (size 1.27 1.27)) hide)
-    )
-    (property "Datasheet" "" (at 148.59 184.15 0)
-      (effects (font (size 1.27 1.27)) hide)
-    )
-    (pin "1")
-    (instances
-      (project "leaf"
-        (path "/e3b58043-16a3-43c8-9fad-9c9784eebfa4/bca9f05a-f031-46a4-95a9-25be55b42bf6"
-          (reference "#PWR022") (unit 1)
-        )
-      )
-    )
-  )
   (symbol (lib_id "Device:R") (at 41.91 116.84 180) (unit 1)
     (in_bom yes) (on_board yes) (dnp no)
@@
         )
       )
-    )
-  )
-  (symbol (lib_id "power:GNDD") (at 135.89 184.15 0) (unit 1)
-    (in_bom yes) (on_board yes) (dnp no) (fields_autoplaced)
-    (property "Reference" "#PWR021" (at 135.89 190.5 0)
-      (effects (font (size 1.27 1.27)) hide)
-    )
-    (property "Value" "GNDD" (at 135.89 187.9045 0)
-      (effects (font (size 1.27 1.27)))
-    )
-    (property "Footprint" "" (at 135.89 184.15 0)
-      (effects (font (size 1.27 1.27)) hide)
-    )
-    (property "Datasheet" "" (at 135.89 184.15 0)
-      (effects (font (size 1.27 1.27)) hide)
-    )
-    (pin "1")
-    (instances
-      (project "leaf"
-        (path "/e3b58043-16a3-43c8-9fad-9c9784eebfa4/bca9f05a-f031-46a4-95a9-25be55b42bf6"
-          (reference "#PWR021") (unit 1)
-        )
-      )
