File: leaf.kicad_sch (KiCad schematic)
At the start: 0 parts

Commit message: updated symbols
Other:
- sheet PMUIO1 ports: added PMIC_INT, PMIC_SLEEP, SoC_I2C0_SCL, SoC_I2C0_SDA; removed none
- sheet Power ports: added PMIC_I2C_SCL, PMIC_I2C_SDA, PMIC_INT, PMIC_SLEEP; removed none
Changed lines of the file:
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@@
+    (stroke (width 0) (type default))
+  )
+  (wire (pts (xy 110.49 106.68) (xy 111.76 106.68))
+    (stroke (width 0) (type default))
+  )
+  (wire (pts (xy 33.02 46.99) (xy 26.67 46.99))
+    (stroke (width 0) (type default))
+  )
+  (wire (pts (xy 33.02 41.91) (xy 26.67 41.91))
+    (stroke (width 0) (type default))
+  )
+  (wire (pts (xy 81.28 111.76) (xy 74.93 111.76))
+    (stroke (width 0) (type default))
+  )
+  (wire (pts (xy 33.02 49.53) (xy 26.67 49.53))
+    (stroke (width 0) (type default))
+  )
+  (wire (pts (xy 33.02 39.37) (xy 26.67 39.37))
+    (stroke (width 0) (type default))
+  )
+  (wire (pts (xy 110.49 104.14) (xy 111.76 104.14))
     (stroke (width 0) (type default))
   )
@@
     (stroke (width 0) (type default))
   )
+  (wire (pts (xy 81.28 109.22) (xy 74.93 109.22))
+    (stroke (width 0) (type default))
+  )
   (wire (pts (xy 77.47 83.82) (xy 81.28 83.82))
     (stroke (width 0) (type default))
@@
     (stroke (width 0) (type default))
   )
-  (wire (pts (xy 114.3 45.72) (xy 124.46 45.72))
+  (wire (pts (xy 116.84 45.72) (xy 127 45.72))
     (stroke (width 0) (type default))
   )
@@
     (stroke (width 0) (type default))
   )
+  (label "PMIC_SLEEP" (at 74.93 111.76 180) (fields_autoplaced)
+    (effects (font (size 1.27 1.27)) (justify right bottom))
+  )
   (label "USB_CTRL" (at 71.12 104.14 0) (fields_autoplaced)
     (effects (font (size 1.27 1.27)) (justify left bottom))
   )
-  (label "USB_CTRL" (at 114.3 45.72 0) (fields_autoplaced)
-    (effects (font (size 1.27 1.27)) (justify left bottom))
+  (label "PMIC_I2C_SCL" (at 111.76 104.14 0) (fields_autoplaced)
+    (effects (font (size 1.27 1.27)) (justify left bottom))
+  )
+  (label "PMIC_I2C_SCL" (at 26.67 46.99 180) (fields_autoplaced)
+    (effects (font (size 1.27 1.27)) (justify right bottom))
+  )
+  (label "PMIC_INT" (at 74.93 109.22 180) (fields_autoplaced)
+    (effects (font (size 1.27 1.27)) (justify right bottom))
+  )
+  (label "PMIC_I2C_SDA" (at 26.67 49.53 180) (fields_autoplaced)
+    (effects (font (size 1.27 1.27)) (justify right bottom))
+  )
+  (label "USB_CTRL" (at 116.84 45.72 0) (fields_autoplaced)
+    (effects (font (size 1.27 1.27)) (justify left bottom))
+  )
+  (label "PMIC_INT" (at 26.67 39.37 180) (fields_autoplaced)
+    (effects (font (size 1.27 1.27)) (justify right bottom))
+  )
+  (label "PMIC_I2C_SDA" (at 111.76 106.68 0) (fields_autoplaced)
+    (effects (font (size 1.27 1.27)) (justify left bottom))
+  )
+  (label "PMIC_SLEEP" (at 26.67 41.91 180) (fields_autoplaced)
+    (effects (font (size 1.27 1.27)) (justify right bottom))
   )
   (sheet (at 81.28 69.85) (size 29.21 17.78) (fields_autoplaced)
@@
       (effects (font (size 1.27 1.27)) (justify left))
     )
+    (pin "PMIC_INT" input (at 81.28 109.22 180)
+      (effects (font (size 1.27 1.27)) (justify left))
+    )
+    (pin "PMIC_SLEEP" output (at 81.28 111.76 180)
+      (effects (font (size 1.27 1.27)) (justify left))
+    )
+    (pin "SoC_I2C0_SCL" output (at 110.49 104.14 0)
+      (effects (font (size 1.27 1.27)) (justify right))
+    )
+    (pin "SoC_I2C0_SDA" bidirectional (at 110.49 106.68 0)
+      (effects (font (size 1.27 1.27)) (justify right))
+    )
     (instances
       (project "leaf"
@@
     )
   )
-  (sheet (at 124.46 97.79) (size 30.48 16.51) (fields_autoplaced)
-    (stroke (width 0.1524) (type solid))
-    (fill (color 0 0 0 0.0000))
-    (property "Sheetname" "Ethernet | PoE" (at 124.46 97.0784 0)
-      (effects (font (size 1.27 1.27)) (justify left bottom))
-    )
-    (property "Sheetfile" "Ethernet.kicad_sch" (at 124.46 114.8846 0)
+  (sheet (at 127 97.79) (size 30.48 16.51) (fields_autoplaced)
+    (stroke (width 0.1524) (type solid))
+    (fill (color 0 0 0 0.0000))
+    (property "Sheetname" "Ethernet | PoE" (at 127 97.0784 0)
+      (effects (font (size 1.27 1.27)) (justify left bottom))
+    )
+    (property "Sheetfile" "Ethernet.kicad_sch" (at 127 114.8846 0)
       (effects (font (size 1.27 1.27)) (justify left top))
     )
@@
     )
   )
-  (sheet (at 124.46 69.85) (size 30.48 17.78) (fields_autoplaced)
-    (stroke (width 0.1524) (type solid))
-    (fill (color 0 0 0 0.0000))
-    (property "Sheetname" "Camera | VCCIO4" (at 124.46 69.1384 0)
-      (effects (font (size 1.27 1.27)) (justify left bottom))
-    )
-    (property "Sheetfile" "Camera.kicad_sch" (at 124.46 88.2146 0)
+  (sheet (at 127 69.85) (size 30.48 17.78) (fields_autoplaced)
+    (stroke (width 0.1524) (type solid))
+    (fill (color 0 0 0 0.0000))
+    (property "Sheetname" "Camera | VCCIO4" (at 127 69.1384 0)
+      (effects (font (size 1.27 1.27)) (justify left bottom))
+    )
+    (property "Sheetfile" "Camera.kicad_sch" (at 127 88.2146 0)
       (effects (font (size 1.27 1.27)) (justify left top))
     )
@@
     )
   )
-  (sheet (at 124.46 35.56) (size 30.48 19.05) (fields_autoplaced)
-    (stroke (width 0.1524) (type solid))
-    (fill (color 0 0 0 0.0000))
-    (property "Sheetname" "USB OTG" (at 124.46 34.8484 0)
-      (effects (font (size 1.27 1.27)) (justify left bottom))
-    )
-    (property "Sheetfile" "USB OTG.kicad_sch" (at 124.46 55.1946 0)
-      (effects (font (size 1.27 1.27)) (justify left top))
-    )
-    (pin "USB_CTRL" input (at 124.46 45.72 180)
+  (sheet (at 127 35.56) (size 30.48 19.05) (fields_autoplaced)
+    (stroke (width 0.1524) (type solid))
+    (fill (color 0 0 0 0.0000))
+    (property "Sheetname" "USB OTG" (at 127 34.8484 0)
+      (effects (font (size 1.27 1.27)) (justify left bottom))
+    )
+    (property "Sheetfile" "USB OTG.kicad_sch" (at 127 55.1946 0)
+      (effects (font (size 1.27 1.27)) (justify left top))
+    )
+    (pin "USB_CTRL" input (at 127 45.72 180)
       (effects (font (size 1.27 1.27)) (justify left))
     )
@@
       (effects (font (size 1.27 1.27)) (justify left top))
     )
-    (instances
+    (pin "PMIC_SLEEP" output (at 33.02 41.91 180)
+      (effects (font (size 1.27 1.27)) (justify left))
+    )
+    (pin "PMIC_INT" input (at 33.02 39.37 180)
+      (effects (font (size 1.27 1.27)) (justify left))
+    )
+    (pin "PMIC_I2C_SCL" input (at 33.02 46.99 180)
+      (effects (font (size 1.27 1.27)) (justify left))
+    )
+    (pin "PMIC_I2C_SDA" bidirectional (at 33.02 49.53 180)
+      (effects (font (size 1.27 1.27)) (justify left))
+    )
+    (instances

Commit message: fix errors
Other:
- sheet Other SoC ports: added RESET; removed none
- sheet PMUIO0 ports: added CLK_32K, RESET; removed none
- sheet Power ports: added PMIC_CLK32K, PMIC_RESET; removed none
Changed lines of the file:
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@@
+    (stroke (width 0) (type default))
+  )
+  (wire (pts (xy 180.34 101.6) (xy 173.99 101.6))
+    (stroke (width 0) (type default))
+  )
+  (wire (pts (xy 62.23 40.64) (xy 68.58 40.64))
+    (stroke (width 0) (type default))
+  )
+  (wire (pts (xy 33.02 111.76) (xy 26.67 111.76))
     (stroke (width 0) (type default))
   )
@@
     (stroke (width 0) (type default))
   )
+  (wire (pts (xy 33.02 107.95) (xy 26.67 107.95))
+    (stroke (width 0) (type default))
+  )
   (wire (pts (xy 110.49 106.68) (xy 111.76 106.68))
     (stroke (width 0) (type default))
@@
     (stroke (width 0) (type default))
   )
+  (wire (pts (xy 33.02 53.34) (xy 26.67 53.34))
+    (stroke (width 0) (type default))
+  )
   (wire (pts (xy 77.47 83.82) (xy 81.28 83.82))
     (stroke (width 0) (type default))
@@
     (effects (font (size 1.27 1.27)) (justify right bottom))
   )
+  (label "PMIC_RESET" (at 26.67 107.95 180) (fields_autoplaced)
+    (effects (font (size 1.27 1.27)) (justify right bottom))
+  )
   (label "USB_CTRL" (at 71.12 104.14 0) (fields_autoplaced)
     (effects (font (size 1.27 1.27)) (justify left bottom))
@@
     (effects (font (size 1.27 1.27)) (justify left bottom))
   )
+  (label "PMIC_CLK32K" (at 68.58 40.64 0) (fields_autoplaced)
+    (effects (font (size 1.27 1.27)) (justify left bottom))
+  )
+  (label "PMIC_RESET" (at 26.67 53.34 180) (fields_autoplaced)
+    (effects (font (size 1.27 1.27)) (justify right bottom))
+  )
   (label "PMIC_I2C_SCL" (at 26.67 46.99 180) (fields_autoplaced)
     (effects (font (size 1.27 1.27)) (justify right bottom))
   )
+  (label "PMIC_CLK32K" (at 26.67 111.76 180) (fields_autoplaced)
+    (effects (font (size 1.27 1.27)) (justify right bottom))
+  )
   (label "PMIC_INT" (at 74.93 109.22 180) (fields_autoplaced)
     (effects (font (size 1.27 1.27)) (justify right bottom))
@@
     (effects (font (size 1.27 1.27)) (justify right bottom))
   )
+  (label "PMIC_RESET" (at 173.99 101.6 180) (fields_autoplaced)
+    (effects (font (size 1.27 1.27)) (justify right bottom))
+  )
   (sheet (at 81.28 69.85) (size 29.21 17.78) (fields_autoplaced)
     (stroke (width 0.1524) (type solid))
@@
       (effects (font (size 1.27 1.27)) (justify left))
     )
+    (pin "RESET" input (at 33.02 107.95 180)
+      (effects (font (size 1.27 1.27)) (justify left))
+    )
+    (pin "CLK_32K" input (at 33.02 111.76 180)
+      (effects (font (size 1.27 1.27)) (justify left))
+    )
     (instances
       (project "leaf"
@@
     )
   )
-  (sheet (at 172.72 97.79) (size 29.21 17.78) (fields_autoplaced)
-    (stroke (width 0.1524) (type solid))
-    (fill (color 0 0 0 0.0000))
-    (property "Sheetname" "Other SoC" (at 172.72 97.0784 0)
-      (effects (font (size 1.27 1.27)) (justify left bottom))
-    )
-    (property "Sheetfile" "OtherSoC.kicad_sch" (at 172.72 116.1546 0)
-      (effects (font (size 1.27 1.27)) (justify left top))
+  (sheet (at 180.34 96.52) (size 29.21 17.78) (fields_autoplaced)
+    (stroke (width 0.1524) (type solid))
+    (fill (color 0 0 0 0.0000))
+    (property "Sheetname" "Other SoC" (at 180.34 95.8084 0)
+      (effects (font (size 1.27 1.27)) (justify left bottom))
+    )
+    (property "Sheetfile" "OtherSoC.kicad_sch" (at 180.34 114.8846 0)
+      (effects (font (size 1.27 1.27)) (justify left top))
+    )
+    (pin "RESET" input (at 180.34 101.6 180)
+      (effects (font (size 1.27 1.27)) (justify left))
     )
     (instances
@@
       (effects (font (size 1.27 1.27)) (justify left))
     )
-    (instances
+    (pin "PMIC_RESET" bidirectional (at 33.02 53.34 180)
+      (effects (font (size 1.27 1.27)) (justify left))
+    )
+    (pin "PMIC_CLK32K" output (at 62.23 40.64 0)
+      (effects (font (size 1.27 1.27)) (justify right))
+    )
+    (instances

Commit message: added OSC, updated annotations
Other:
- added sheet SoC OSC_PLL (SoC_OSC_PLL.kicad_sch)
- sheet Other SoC ports: added none; removed RESET
Changed lines of the file:
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@@
     (company "Qingdao IotPi Information Technology")
   )
+  (wire (pts (xy 31.75 140.97) (xy 25.4 140.97))
+    (stroke (width 0) (type default))
+  )
   (wire (pts (xy 71.12 104.14) (xy 81.28 104.14))
     (stroke (width 0) (type default))
   )
-  (wire (pts (xy 180.34 101.6) (xy 173.99 101.6))
-    (stroke (width 0) (type default))
-  )
   (wire (pts (xy 62.23 40.64) (xy 68.58 40.64))
     (stroke (width 0) (type default))
@@
     (stroke (width 0) (type default))
   )
-  (wire (pts (xy 116.84 45.72) (xy 127 45.72))
+  (wire (pts (xy 129.54 45.72) (xy 139.7 45.72))
     (stroke (width 0) (type default))
   )
@@
     (effects (font (size 1.27 1.27)) (justify right bottom))
   )
-  (label "USB_CTRL" (at 116.84 45.72 0) (fields_autoplaced)
+  (label "USB_CTRL" (at 129.54 45.72 0) (fields_autoplaced)
     (effects (font (size 1.27 1.27)) (justify left bottom))
   )
@@
     (effects (font (size 1.27 1.27)) (justify right bottom))
   )
-  (label "PMIC_RESET" (at 173.99 101.6 180) (fields_autoplaced)
+  (label "PMIC_RESET" (at 25.4 140.97 180) (fields_autoplaced)
     (effects (font (size 1.27 1.27)) (justify right bottom))
   )
@@
       (effects (font (size 1.27 1.27)) (justify left top))
     )
-    (pin "RESET" input (at 180.34 101.6 180)
-      (effects (font (size 1.27 1.27)) (justify left))
-    )
     (instances
       (project "leaf"
         (path "/e3b58043-16a3-43c8-9fad-9c9784eebfa4" (page "23"))
+      )
+    )
+  )
+  (sheet (at 31.75 135.89) (size 31.75 17.78) (fields_autoplaced)
+    (stroke (width 0.1524) (type solid))
+    (fill (color 0 0 0 0.0000))
+    (property "Sheetname" "SoC OSC_PLL" (at 31.75 135.1784 0)
+      (effects (font (size 1.27 1.27)) (justify left bottom))
+    )
+    (property "Sheetfile" "SoC_OSC_PLL.kicad_sch" (at 31.75 154.2546 0)
+      (effects (font (size 1.27 1.27)) (justify left top))
+    )
+    (pin "RESET" input (at 31.75 140.97 180)
+      (effects (font (size 1.27 1.27)) (justify left))
+    )
+    (instances
+      (project "leaf"
+        (path "/e3b58043-16a3-43c8-9fad-9c9784eebfa4" (page "24"))
       )
     )
@@
     )
   )
-  (sheet (at 81.28 35.56) (size 29.21 19.05) (fields_autoplaced)
-    (stroke (width 0.1524) (type solid))
-    (fill (color 0 0 0 0.0000))
-    (property "Sheetname" "DDR" (at 81.28 34.8484 0)
-      (effects (font (size 1.27 1.27)) (justify left bottom))
-    )
-    (property "Sheetfile" "DDR.kicad_sch" (at 81.28 55.1946 0)
+  (sheet (at 90.17 35.56) (size 29.21 19.05) (fields_autoplaced)
+    (stroke (width 0.1524) (type solid))
+    (fill (color 0 0 0 0.0000))
+    (property "Sheetname" "DDR" (at 90.17 34.8484 0)
+      (effects (font (size 1.27 1.27)) (justify left bottom))
+    )
+    (property "Sheetfile" "DDR.kicad_sch" (at 90.17 55.1946 0)
       (effects (font (size 1.27 1.27)) (justify left top))
     )
@@
     )
   )
-  (sheet (at 172.72 35.56) (size 29.21 19.05) (fields_autoplaced)
-    (stroke (width 0.1524) (type solid))
-    (fill (color 0 0 0 0.0000))
-    (property "Sheetname" "Display" (at 172.72 34.8484 0)
-      (effects (font (size 1.27 1.27)) (justify left bottom))
-    )
-    (property "Sheetfile" "Display.kicad_sch" (at 172.72 55.1946 0)
+  (sheet (at 180.34 35.56) (size 29.21 19.05) (fields_autoplaced)
+    (stroke (width 0.1524) (type solid))
+    (fill (color 0 0 0 0.0000))
+    (property "Sheetname" "Display" (at 180.34 34.8484 0)
+      (effects (font (size 1.27 1.27)) (justify left bottom))
+    )
+    (property "Sheetfile" "Display.kicad_sch" (at 180.34 55.1946 0)
       (effects (font (size 1.27 1.27)) (justify left top))
     )
@@
     )
   )
-  (sheet (at 127 35.56) (size 30.48 19.05) (fields_autoplaced)
-    (stroke (width 0.1524) (type solid))
-    (fill (color 0 0 0 0.0000))
-    (property "Sheetname" "USB OTG" (at 127 34.8484 0)
-      (effects (font (size 1.27 1.27)) (justify left bottom))
-    )
-    (property "Sheetfile" "USB OTG.kicad_sch" (at 127 55.1946 0)
-      (effects (font (size 1.27 1.27)) (justify left top))
-    )
-    (pin "USB_CTRL" input (at 127 45.72 180)
+  (sheet (at 139.7 35.56) (size 30.48 19.05) (fields_autoplaced)
+    (stroke (width 0.1524) (type solid))
+    (fill (color 0 0 0 0.0000))
+    (property "Sheetname" "USB OTG" (at 139.7 34.8484 0)
+      (effects (font (size 1.27 1.27)) (justify left bottom))
+    )
+    (property "Sheetfile" "USB OTG.kicad_sch" (at 139.7 55.1946 0)
+      (effects (font (size 1.27 1.27)) (justify left top))
+    )
+    (pin "USB_CTRL" input (at 139.7 45.72 180)
       (effects (font (size 1.27 1.27)) (justify left))
     )
@@
     )
   )
-  (sheet (at 172.72 69.85) (size 29.21 17.78) (fields_autoplaced)
-    (stroke (width 0.1524) (type solid))
-    (fill (color 0 0 0 0.0000))
-    (property "Sheetname" "WiFi" (at 172.72 69.1384 0)
-      (effects (font (size 1.27 1.27)) (justify left bottom))
-    )
-    (property "Sheetfile" "WiFi.kicad_sch" (at 172.72 88.2146 0)
-      (effects (font (size 1.27 1.27)) (justify left top))
-    )
+  (sheet (at 180.34 69.85) (size 29.21 17.78) (fields_autoplaced)
+    (stroke (width 0.1524) (type solid))
+    (fill (color 0 0 0 0.0000))
+    (property "Sheetname" "WiFi" (at 180.34 69.1384 0)
+      (effects (font (size 1.27 1.27)) (justify left bottom))
+    )
+    (property "Sheetfile" "WiFi.kicad_sch" (at 180.34 88.2146 0)
+      (effects (font (size 1.27 1.27)) (justify left top))
+    )
