File: DDR_Chips.kicad_sch (KiCad schematic)
At the start: 1 part

Commit message: remove DDR decoupling capacitors sheets
Other:
- removed sheet DDR Filter Capacitors
Changed lines of the file:
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@@
-    (stroke (width 0) (type default))
-  )
-  (wire (pts (xy 35.56 172.72) (xy 43.18 172.72))
     (stroke (width 0) (type default))
   )
@@
   (label "DDR4_D22" (at 148.59 99.06 0) (fields_autoplaced)
     (effects (font (size 1.27 1.27)) (justify left bottom))
-  )
-  (label "VCC2V5_DDR" (at 35.56 172.72 180) (fields_autoplaced)
-    (effects (font (size 1.27 1.27)) (justify right bottom))
   )
   (label "DDR4_D10" (at 245.11 31.75 0) (fields_autoplaced)
@@
       )
     )
-  )
-  (sheet (at 43.18 157.48) (size 45.72 26.67) (fields_autoplaced)
-    (stroke (width 0.1524) (type solid))
-    (fill (color 0 0 0 0.0000))
-    (property "Sheetname" "DDR Filter Capacitors" (at 43.18 156.7684 0)
-      (effects (font (size 1.27 1.27)) (justify left bottom))
-    )
-    (property "Sheetfile" "DDR_filter_capacitors.kicad_sch" (at 43.18 184.7346 0)
-      (effects (font (size 1.27 1.27)) (justify left top))
-    )
-    (pin "VCC25_DDR" input (at 43.18 172.72 180)
-      (effects (font (size 1.27 1.27)) (justify left))
-    )
-    (instances
-      (project "leaf"
-        (path "/e3b58043-16a3-43c8-9fad-9c9784eebfa4/9453ad46-b3ff-4d4e-8aa6-7cc75aa0f522/43b336b1-9a2a-4a37-8b6d-a408b4dd9ca2" (page "19"))
-      )
-    )
