File: DDR_Chips.kicad_sch (KiCad schematic)
At the start: 13 parts

Commit message: updated annotations
Parts:
- renumbered RN5 to RN4, RN4 to RN5
Changed lines of the file:
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@@
         )
         (path "/e3b58043-16a3-43c8-9fad-9c9784eebfa4/9453ad46-b3ff-4d4e-8aa6-7cc75aa0f522/43b336b1-9a2a-4a37-8b6d-a408b4dd9ca2"
-          (reference "C109") (unit 1)
+          (reference "C126") (unit 1)
         )
         (path "/e3b58043-16a3-43c8-9fad-9c9784eebfa4/9453ad46-b3ff-4d4e-8aa6-7cc75aa0f522/43b336b1-9a2a-4a37-8b6d-a408b4dd9ca2/c5996722-c916-43bd-91c1-647d75e652e6"
@@
         )
         (path "/e3b58043-16a3-43c8-9fad-9c9784eebfa4/9453ad46-b3ff-4d4e-8aa6-7cc75aa0f522/43b336b1-9a2a-4a37-8b6d-a408b4dd9ca2"
-          (reference "R70") (unit 1)
+          (reference "R65") (unit 1)
         )
         (path "/e3b58043-16a3-43c8-9fad-9c9784eebfa4/9453ad46-b3ff-4d4e-8aa6-7cc75aa0f522/43b336b1-9a2a-4a37-8b6d-a408b4dd9ca2/c5996722-c916-43bd-91c1-647d75e652e6"
@@
         )
         (path "/e3b58043-16a3-43c8-9fad-9c9784eebfa4/9453ad46-b3ff-4d4e-8aa6-7cc75aa0f522/43b336b1-9a2a-4a37-8b6d-a408b4dd9ca2"
-          (reference "R58") (unit 1)
+          (reference "R61") (unit 1)
         )
         (path "/e3b58043-16a3-43c8-9fad-9c9784eebfa4/9453ad46-b3ff-4d4e-8aa6-7cc75aa0f522/43b336b1-9a2a-4a37-8b6d-a408b4dd9ca2/c5996722-c916-43bd-91c1-647d75e652e6"
@@
         )
         (path "/e3b58043-16a3-43c8-9fad-9c9784eebfa4/9453ad46-b3ff-4d4e-8aa6-7cc75aa0f522/43b336b1-9a2a-4a37-8b6d-a408b4dd9ca2"
-          (reference "R68") (unit 1)
+          (reference "R64") (unit 1)
         )
         (path "/e3b58043-16a3-43c8-9fad-9c9784eebfa4/9453ad46-b3ff-4d4e-8aa6-7cc75aa0f522/43b336b1-9a2a-4a37-8b6d-a408b4dd9ca2/c5996722-c916-43bd-91c1-647d75e652e6"
@@
         )
         (path "/e3b58043-16a3-43c8-9fad-9c9784eebfa4/9453ad46-b3ff-4d4e-8aa6-7cc75aa0f522/43b336b1-9a2a-4a37-8b6d-a408b4dd9ca2"
-          (reference "R69") (unit 1)
+          (reference "R63") (unit 1)
         )
         (path "/e3b58043-16a3-43c8-9fad-9c9784eebfa4/9453ad46-b3ff-4d4e-8aa6-7cc75aa0f522/43b336b1-9a2a-4a37-8b6d-a408b4dd9ca2/c5996722-c916-43bd-91c1-647d75e652e6"
@@
         )
         (path "/e3b58043-16a3-43c8-9fad-9c9784eebfa4/9453ad46-b3ff-4d4e-8aa6-7cc75aa0f522/43b336b1-9a2a-4a37-8b6d-a408b4dd9ca2"
-          (reference "R67") (unit 1)
+          (reference "R62") (unit 1)
         )
         (path "/e3b58043-16a3-43c8-9fad-9c9784eebfa4/9453ad46-b3ff-4d4e-8aa6-7cc75aa0f522/43b336b1-9a2a-4a37-8b6d-a408b4dd9ca2/c5996722-c916-43bd-91c1-647d75e652e6"
@@
   (symbol (lib_id "Device:R_Pack04") (at 93.98 166.37 270) (unit 1)
     (in_bom yes) (on_board yes) (dnp no) (fields_autoplaced)
-    (property "Reference" "RN5" (at 93.98 154.94 90)
+    (property "Reference" "RN4" (at 93.98 154.94 90)
       (effects (font (size 1.27 1.27)))
     )
@@
       (project "leaf"
         (path "/e3b58043-16a3-43c8-9fad-9c9784eebfa4/9453ad46-b3ff-4d4e-8aa6-7cc75aa0f522/43b336b1-9a2a-4a37-8b6d-a408b4dd9ca2"
-          (reference "RN5") (unit 1)
+          (reference "RN4") (unit 1)
         )
       )
@@
         )
         (path "/e3b58043-16a3-43c8-9fad-9c9784eebfa4/9453ad46-b3ff-4d4e-8aa6-7cc75aa0f522/43b336b1-9a2a-4a37-8b6d-a408b4dd9ca2"
-          (reference "R57") (unit 1)
+          (reference "R60") (unit 1)
         )
         (path "/e3b58043-16a3-43c8-9fad-9c9784eebfa4/9453ad46-b3ff-4d4e-8aa6-7cc75aa0f522/43b336b1-9a2a-4a37-8b6d-a408b4dd9ca2/c5996722-c916-43bd-91c1-647d75e652e6"
@@
         )
         (path "/e3b58043-16a3-43c8-9fad-9c9784eebfa4/9453ad46-b3ff-4d4e-8aa6-7cc75aa0f522/43b336b1-9a2a-4a37-8b6d-a408b4dd9ca2"
-          (reference "#PWR0111") (unit 1)
+          (reference "#PWR0124") (unit 1)
         )
         (path "/e3b58043-16a3-43c8-9fad-9c9784eebfa4/9453ad46-b3ff-4d4e-8aa6-7cc75aa0f522/43b336b1-9a2a-4a37-8b6d-a408b4dd9ca2/c5996722-c916-43bd-91c1-647d75e652e6"
@@
   (symbol (lib_id "Device:R_Pack04") (at 41.91 184.15 270) (unit 1)
     (in_bom yes) (on_board yes) (dnp no) (fields_autoplaced)
-    (property "Reference" "RN4" (at 41.91 172.72 90)
+    (property "Reference" "RN5" (at 41.91 172.72 90)
       (effects (font (size 1.27 1.27)))
     )
@@
       (project "leaf"
         (path "/e3b58043-16a3-43c8-9fad-9c9784eebfa4/9453ad46-b3ff-4d4e-8aa6-7cc75aa0f522/43b336b1-9a2a-4a37-8b6d-a408b4dd9ca2"
-          (reference "RN4") (unit 1)
+          (reference "RN5") (unit 1)
         )
       )
@@
     (instances
       (project "leaf"
-        (path "/e3b58043-16a3-43c8-9fad-9c9784eebfa4/9453ad46-b3ff-4d4e-8aa6-7cc75aa0f522/43b336b1-9a2a-4a37-8b6d-a408b4dd9ca2" (page "17"))
-      )
-    )
+        (path "/e3b58043-16a3-43c8-9fad-9c9784eebfa4/9453ad46-b3ff-4d4e-8aa6-7cc75aa0f522/43b336b1-9a2a-4a37-8b6d-a408b4dd9ca2" (page "26"))
+      )
+    )
