File: PMUIO1.kicad_sch (KiCad schematic)
At the start: 2 parts, among them U1 rv1126/rv1109

Commit message: updated symbols
Connections:
- net SoC_I2C0_SCL: now reaches U1.AA7 (I2C0_SCL/GPIO0_B4_u)
- net PMIC_INT: now reaches U1.W10 (PMIC_INT/PWM7_IR_M0/GPIO0_B1_d)
- net PMIC_SLEEP: now reaches U1.Y10 (PMIC_SLEEP/TSADC_SHUT_M1/PWM6_M0/GPIO0_B2_d)
- net SoC_I2C0_SDA: now reaches U1.Y7 (I2C0_SDA/GPIO0_B5_u)
- no-connect marks 9 -> 5
Changed lines of the file:
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@@
   (junction (at 151.13 105.41) (diameter 0) (color 0 0 0 0)
   )
-  (no_connect (at 133.35 67.31))
   (no_connect (at 133.35 95.25))
   (no_connect (at 133.35 76.2))
   (no_connect (at 133.35 73.66))
   (no_connect (at 133.35 97.79))
-  (no_connect (at 133.35 80.01))
   (no_connect (at 133.35 90.17))
-  (no_connect (at 133.35 82.55))
-  (no_connect (at 133.35 69.85))
+  (wire (pts (xy 39.37 39.37) (xy 45.72 39.37))
+    (stroke (width 0) (type default))
+  )
   (wire (pts (xy 39.37 34.29) (xy 64.77 34.29))
     (stroke (width 0) (type default))
@@
     (stroke (width 0) (type default))
   )
+  (wire (pts (xy 39.37 48.26) (xy 45.72 48.26))
+    (stroke (width 0) (type default))
+  )
   (wire (pts (xy 133.35 105.41) (xy 151.13 105.41))
     (stroke (width 0) (type default))
   )
+  (wire (pts (xy 133.35 82.55) (xy 139.7 82.55))
+    (stroke (width 0) (type default))
+  )
+  (wire (pts (xy 133.35 69.85) (xy 139.7 69.85))
+    (stroke (width 0) (type default))
+  )
+  (wire (pts (xy 133.35 80.01) (xy 139.7 80.01))
+    (stroke (width 0) (type default))
+  )
+  (wire (pts (xy 133.35 67.31) (xy 139.7 67.31))
+    (stroke (width 0) (type default))
+  )
   (wire (pts (xy 151.13 105.41) (xy 158.75 105.41))
     (stroke (width 0) (type default))
@@
     (stroke (width 0) (type default))
   )
+  (wire (pts (xy 39.37 41.91) (xy 45.72 41.91))
+    (stroke (width 0) (type default))
+  )
+  (wire (pts (xy 39.37 45.72) (xy 45.72 45.72))
+    (stroke (width 0) (type default))
+  )
   (text "USB_CTRL must use GPIO0_C1_d / AA4" (at 172.72 86.36 0)
     (effects (font (size 1.27 1.27)) (justify left bottom))
@@
     (effects (font (size 1.27 1.27)) (justify left bottom))
   )
+  (label "PMIC_INT" (at 45.72 39.37 0) (fields_autoplaced)
+    (effects (font (size 1.27 1.27)) (justify left bottom))
+  )
+  (label "PMIC_SLEEP" (at 45.72 41.91 0) (fields_autoplaced)
+    (effects (font (size 1.27 1.27)) (justify left bottom))
+  )
   (label "USB_CTRL" (at 158.75 86.36 0) (fields_autoplaced)
     (effects (font (size 1.27 1.27)) (justify left bottom))
   )
+  (label "SoC_I2C0_SDA" (at 45.72 48.26 0) (fields_autoplaced)
+    (effects (font (size 1.27 1.27)) (justify left bottom))
+  )
+  (label "SoC_I2C0_SCL" (at 45.72 45.72 0) (fields_autoplaced)
+    (effects (font (size 1.27 1.27)) (justify left bottom))
+  )
   (label "VCC3V3_SYS" (at 158.75 105.41 0) (fields_autoplaced)
     (effects (font (size 1.27 1.27)) (justify left bottom))
   )
   (label "VCC3V3_SYS" (at 64.77 27.94 0) (fields_autoplaced)
+    (effects (font (size 1.27 1.27)) (justify left bottom))
+  )
+  (label "SoC_I2C0_SCL" (at 139.7 67.31 0) (fields_autoplaced)
+    (effects (font (size 1.27 1.27)) (justify left bottom))
+  )
+  (label "SoC_I2C0_SDA" (at 139.7 69.85 0) (fields_autoplaced)
+    (effects (font (size 1.27 1.27)) (justify left bottom))
+  )
+  (label "PMIC_INT" (at 139.7 80.01 0) (fields_autoplaced)
+    (effects (font (size 1.27 1.27)) (justify left bottom))
+  )
+  (label "PMIC_SLEEP" (at 139.7 82.55 0) (fields_autoplaced)
     (effects (font (size 1.27 1.27)) (justify left bottom))
   )
@@
     )
   )
+  (hierarchical_label "PMIC_SLEEP" (shape output) (at 39.37 41.91 180) (fields_autoplaced)
+    (effects (font (size 1.27 1.27)) (justify right))
+  )
+  (hierarchical_label "PMIC_INT" (shape input) (at 39.37 39.37 180) (fields_autoplaced)
+    (effects (font (size 1.27 1.27)) (justify right))
+  )
   (hierarchical_label "FLASH_VOL_SEL" (shape input) (at 39.37 34.29 180) (fields_autoplaced)
     (effects (font (size 1.27 1.27)) (justify right))
   )
   (hierarchical_label "USB_CTRL" (shape output) (at 39.37 24.13 180) (fields_autoplaced)
+    (effects (font (size 1.27 1.27)) (justify right))
+  )
+  (hierarchical_label "SoC_I2C0_SCL" (shape output) (at 39.37 45.72 180) (fields_autoplaced)
+    (effects (font (size 1.27 1.27)) (justify right))
+  )
+  (hierarchical_label "SoC_I2C0_SDA" (shape bidirectional) (at 39.37 48.26 180) (fields_autoplaced)
     (effects (font (size 1.27 1.27)) (justify right))
   )
@@
     (pin "E20")
     (pin "F19")
-    (pin "F19")
     (pin "F20")

Commit message: added OSC, updated annotations
Parts:
- renumbered U1 to U3001
Changed lines of the file:
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@@
         )
         (path "/e3b58043-16a3-43c8-9fad-9c9784eebfa4/74154bd6-827c-4e46-8351-0d1a22db546e"
-          (reference "C136") (unit 1)
+          (reference "C20001") (unit 1)
         )
       )
@@
   (symbol (lib_id "CPU_Rockchip:rv1126_rv1109") (at 93.98 81.28 0) (unit 5)
     (in_bom yes) (on_board yes) (dnp no) (fields_autoplaced)
-    (property "Reference" "U1" (at 92.71 52.9971 0)
+    (property "Reference" "U3001" (at 92.71 52.9971 0)
       (effects (font (size 1.27 1.27)))
     )
@@
       (project "leaf"
         (path "/e3b58043-16a3-43c8-9fad-9c9784eebfa4/74154bd6-827c-4e46-8351-0d1a22db546e"
-          (reference "U1") (unit 5)
+          (reference "U3001") (unit 5)
         )
       )
@@
   (symbol (lib_id "power:GND") (at 151.13 123.19 0) (unit 1)
     (in_bom yes) (on_board yes) (dnp no) (fields_autoplaced)
-    (property "Reference" "#PWR0127" (at 151.13 129.54 0)
+    (property "Reference" "#PWR020001" (at 151.13 129.54 0)
       (effects (font (size 1.27 1.27)) hide)
     )
@@
       (project "leaf"
         (path "/e3b58043-16a3-43c8-9fad-9c9784eebfa4/74154bd6-827c-4e46-8351-0d1a22db546e"
-          (reference "#PWR0127") (unit 1)
+          (reference "#PWR020001") (unit 1)
         )
       )

Commit message: move DDR power decoupling capacitors into DDR4 Sheet
Parts:
- renumbered U3001 to U2
Changed lines of the file:
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@@
         )
         (path "/e3b58043-16a3-43c8-9fad-9c9784eebfa4/74154bd6-827c-4e46-8351-0d1a22db546e"
-          (reference "C20001") (unit 1)
+          (reference "C137") (unit 1)
         )
       )
@@
   (symbol (lib_id "CPU_Rockchip:rv1126_rv1109") (at 93.98 81.28 0) (unit 5)
     (in_bom yes) (on_board yes) (dnp no) (fields_autoplaced)
-    (property "Reference" "U3001" (at 92.71 52.9971 0)
+    (property "Reference" "U2" (at 92.71 52.9971 0)
       (effects (font (size 1.27 1.27)))
     )
@@
       (project "leaf"
         (path "/e3b58043-16a3-43c8-9fad-9c9784eebfa4/74154bd6-827c-4e46-8351-0d1a22db546e"
-          (reference "U3001") (unit 5)
+          (reference "U2") (unit 5)
         )
       )
@@
   (symbol (lib_id "power:GND") (at 151.13 123.19 0) (unit 1)
     (in_bom yes) (on_board yes) (dnp no) (fields_autoplaced)
-    (property "Reference" "#PWR020001" (at 151.13 129.54 0)
+    (property "Reference" "#PWR0120" (at 151.13 129.54 0)
       (effects (font (size 1.27 1.27)) hide)
     )
@@
       (project "leaf"
         (path "/e3b58043-16a3-43c8-9fad-9c9784eebfa4/74154bd6-827c-4e46-8351-0d1a22db546e"
-          (reference "#PWR020001") (unit 1)
+          (reference "#PWR0120") (unit 1)
         )
       )
