File: Power.kicad_sch (KiCad schematic)
At the start: 13 parts, among them U9 BL8039

Commit message: fixing warnings
Other:
- moved on the sheet: NT1

Commit message: fix ERC warnings
Parts:
- NT1: footprint (none) -> NetTie:NetTie-3_SMD_Pad2.0mm
Changed lines of the file:
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@@
       (effects (font (size 1.27 1.27)))
     )
-    (property "Footprint" "" (at 260.35 43.18 0)
+    (property "Footprint" "NetTie:NetTie-3_SMD_Pad2.0mm" (at 260.35 43.18 0)
       (effects (font (size 1.27 1.27)) hide)
     )

Commit message: added OSC, updated annotations
Parts:
- renumbered U9 to U2001
Changed lines of the file:
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@@
   (symbol (lib_id "Leaf_Converter_DCDC:BL8039") (at 86.36 97.79 0) (unit 1)
     (in_bom yes) (on_board yes) (dnp no) (fields_autoplaced)
-    (property "Reference" "U9" (at 88.9 92.3671 0)
+    (property "Reference" "U2001" (at 88.9 92.3671 0)
       (effects (font (size 1.27 1.27)))
     )
@@
       (project "leaf"
         (path "/e3b58043-16a3-43c8-9fad-9c9784eebfa4/cc9fb3ac-19c3-47a8-ba7d-678b4d514ff0"
-          (reference "U9") (unit 1)
+          (reference "U2001") (unit 1)
         )
       )
@@
         )
         (path "/e3b58043-16a3-43c8-9fad-9c9784eebfa4/cc9fb3ac-19c3-47a8-ba7d-678b4d514ff0"
-          (reference "#PWR032") (unit 1)
+          (reference "#PWR02011") (unit 1)
         )
       )
@@
         )
         (path "/e3b58043-16a3-43c8-9fad-9c9784eebfa4/cc9fb3ac-19c3-47a8-ba7d-678b4d514ff0"
-          (reference "#PWR031") (unit 1)
+          (reference "#PWR02010") (unit 1)
         )
       )
@@
         )
         (path "/e3b58043-16a3-43c8-9fad-9c9784eebfa4/cc9fb3ac-19c3-47a8-ba7d-678b4d514ff0"
-          (reference "C152") (unit 1)
+          (reference "C2002") (unit 1)
         )
       )
@@
   (symbol (lib_id "power:GND") (at 200.66 49.53 0) (unit 1)
     (in_bom yes) (on_board yes) (dnp no) (fields_autoplaced)
-    (property "Reference" "#PWR0143" (at 200.66 55.88 0)
+    (property "Reference" "#PWR02006" (at 200.66 55.88 0)
       (effects (font (size 1.27 1.27)) hide)
     )
@@
       (project "leaf"
         (path "/e3b58043-16a3-43c8-9fad-9c9784eebfa4/cc9fb3ac-19c3-47a8-ba7d-678b4d514ff0"
-          (reference "#PWR0143") (unit 1)
+          (reference "#PWR02006") (unit 1)
         )
       )
@@
         )
         (path "/e3b58043-16a3-43c8-9fad-9c9784eebfa4/cc9fb3ac-19c3-47a8-ba7d-678b4d514ff0"
-          (reference "C153") (unit 1)
+          (reference "C2004") (unit 1)
         )
       )
@@
         )
         (path "/e3b58043-16a3-43c8-9fad-9c9784eebfa4/cc9fb3ac-19c3-47a8-ba7d-678b4d514ff0"
-          (reference "R78") (unit 1)
+          (reference "R2002") (unit 1)
         )
       )
@@
         )
         (path "/e3b58043-16a3-43c8-9fad-9c9784eebfa4/cc9fb3ac-19c3-47a8-ba7d-678b4d514ff0"
-          (reference "C156") (unit 1)
+          (reference "C2003") (unit 1)
         )
       )
@@
   (symbol (lib_id "power:GNDA") (at 74.93 124.46 0) (unit 1)
     (in_bom yes) (on_board yes) (dnp no) (fields_autoplaced)
-    (property "Reference" "#PWR0145" (at 74.93 130.81 0)
+    (property "Reference" "#PWR02002" (at 74.93 130.81 0)
       (effects (font (size 1.27 1.27)) hide)
     )
@@
       (project "leaf"
         (path "/e3b58043-16a3-43c8-9fad-9c9784eebfa4/cc9fb3ac-19c3-47a8-ba7d-678b4d514ff0"
-          (reference "#PWR0145") (unit 1)
+          (reference "#PWR02002") (unit 1)
         )
       )
@@
         )
         (path "/e3b58043-16a3-43c8-9fad-9c9784eebfa4/cc9fb3ac-19c3-47a8-ba7d-678b4d514ff0"
-          (reference "L7") (unit 1)
+          (reference "L2001") (unit 1)
         )
       )
@@
   (symbol (lib_id "power:PWR_FLAG") (at 234.95 43.18 0) (unit 1)
     (in_bom yes) (on_board yes) (dnp no) (fields_autoplaced)
-    (property "Reference" "#FLG017" (at 234.95 41.275 0)
+    (property "Reference" "#FLG02005" (at 234.95 41.275 0)
       (effects (font (size 1.27 1.27)) hide)
     )
@@
       (project "leaf"
         (path "/e3b58043-16a3-43c8-9fad-9c9784eebfa4/cc9fb3ac-19c3-47a8-ba7d-678b4d514ff0"
-          (reference "#FLG017") (unit 1)
+          (reference "#FLG02005") (unit 1)
         )
       )
@@
         )
         (path "/e3b58043-16a3-43c8-9fad-9c9784eebfa4/cc9fb3ac-19c3-47a8-ba7d-678b4d514ff0"
-          (reference "C154") (unit 1)
+          (reference "C2005") (unit 1)
         )
       )
@@
   (symbol (lib_id "power:GNDA") (at 43.18 111.76 0) (unit 1)
     (in_bom yes) (on_board yes) (dnp no) (fields_autoplaced)
-    (property "Reference" "#PWR0144" (at 43.18 118.11 0)
+    (property "Reference" "#PWR02001" (at 43.18 118.11 0)
       (effects (font (size 1.27 1.27)) hide)
     )
@@
       (project "leaf"
         (path "/e3b58043-16a3-43c8-9fad-9c9784eebfa4/cc9fb3ac-19c3-47a8-ba7d-678b4d514ff0"
-          (reference "#PWR0144") (unit 1)
+          (reference "#PWR02001") (unit 1)
         )
       )
@@
         )
         (path "/e3b58043-16a3-43c8-9fad-9c9784eebfa4/cc9fb3ac-19c3-47a8-ba7d-678b4d514ff0"
-          (reference "#PWR020") (unit 1)
+          (reference "#PWR02007") (unit 1)
         )
       )
@@
         )
         (path "/e3b58043-16a3-43c8-9fad-9c9784eebfa4/cc9fb3ac-19c3-47a8-ba7d-678b4d514ff0"
-          (reference "R76") (unit 1)
+          (reference "R2003") (unit 1)
         )
       )
@@
   (symbol (lib_id "power:GNDA") (at 88.9 124.46 0) (unit 1)
     (in_bom yes) (on_board yes) (dnp no) (fields_autoplaced)
-    (property "Reference" "#PWR0146" (at 88.9 130.81 0)
+    (property "Reference" "#PWR02003" (at 88.9 130.81 0)
       (effects (font (size 1.27 1.27)) hide)
     )
@@
       (project "leaf"
         (path "/e3b58043-16a3-43c8-9fad-9c9784eebfa4/cc9fb3ac-19c3-47a8-ba7d-678b4d514ff0"
-          (reference "#PWR0146") (unit 1)
+          (reference "#PWR02003") (unit 1)
         )
       )
@@
         )
         (path "/e3b58043-16a3-43c8-9fad-9c9784eebfa4/cc9fb3ac-19c3-47a8-ba7d-678b4d514ff0"
-          (reference "C155") (unit 1)
+          (reference "C2006") (unit 1)
         )
       )
@@
   (symbol (lib_id "power:PWR_FLAG") (at 185.42 44.45 0) (unit 1)
     (in_bom yes) (on_board yes) (dnp no) (fields_autoplaced)
-    (property "Reference" "#FLG01" (at 185.42 42.545 0)
+    (property "Reference" "#FLG02002" (at 185.42 42.545 0)
       (effects (font (size 1.27 1.27)) hide)
     )
@@
       (project "leaf"
         (path "/e3b58043-16a3-43c8-9fad-9c9784eebfa4/cc9fb3ac-19c3-47a8-ba7d-678b4d514ff0"
-          (reference "#FLG01") (unit 1)
+          (reference "#FLG02002") (unit 1)
         )
       )
@@
         )
         (path "/e3b58043-16a3-43c8-9fad-9c9784eebfa4/cc9fb3ac-19c3-47a8-ba7d-678b4d514ff0"
-          (reference "C151") (unit 1)
+          (reference "C2001") (unit 1)
         )
       )
@@
         )
         (path "/e3b58043-16a3-43c8-9fad-9c9784eebfa4/cc9fb3ac-19c3-47a8-ba7d-678b4d514ff0"
-          (reference "#PWR030") (unit 1)
+          (reference "#PWR02009") (unit 1)
         )
       )
@@
         )
         (path "/e3b58043-16a3-43c8-9fad-9c9784eebfa4/cc9fb3ac-19c3-47a8-ba7d-678b4d514ff0"
-          (reference "R75") (unit 1)
+          (reference "R2001") (unit 1)
         )
       )
@@
   (symbol (lib_id "power:GNDA") (at 166.37 154.94 90) (unit 1)
     (in_bom yes) (on_board yes) (dnp no) (fields_autoplaced)
-    (property "Reference" "#PWR0148" (at 172.72 154.94 0)
+    (property "Reference" "#PWR02004" (at 172.72 154.94 0)
       (effects (font (size 1.27 1.27)) hide)
     )
@@
       (project "leaf"
         (path "/e3b58043-16a3-43c8-9fad-9c9784eebfa4/cc9fb3ac-19c3-47a8-ba7d-678b4d514ff0"
-          (reference "#PWR0148") (unit 1)
+          (reference "#PWR02004") (unit 1)
         )
       )
@@
         )
         (path "/e3b58043-16a3-43c8-9fad-9c9784eebfa4/cc9fb3ac-19c3-47a8-ba7d-678b4d514ff0"
-          (reference "R77") (unit 1)
+          (reference "R2004") (unit 1)
         )
       )
@@
   (symbol (lib_id "power:PWR_FLAG") (at 220.98 43.18 0) (unit 1)
     (in_bom yes) (on_board yes) (dnp no) (fields_autoplaced)
-    (property "Reference" "#FLG07" (at 220.98 41.275 0)
+    (property "Reference" "#FLG02004" (at 220.98 41.275 0)
       (effects (font (size 1.27 1.27)) hide)
     )
@@
       (project "leaf"
         (path "/e3b58043-16a3-43c8-9fad-9c9784eebfa4/cc9fb3ac-19c3-47a8-ba7d-678b4d514ff0"
-          (reference "#FLG07") (unit 1)
+          (reference "#FLG02004") (unit 1)
         )
       )
@@
   (symbol (lib_id "power:PWR_FLAG") (at 205.74 43.18 0) (unit 1)
     (in_bom yes) (on_board yes) (dnp no) (fields_autoplaced)
-    (property "Reference" "#FLG02" (at 205.74 41.275 0)
+    (property "Reference" "#FLG02003" (at 205.74 41.275 0)
       (effects (font (size 1.27 1.27)) hide)
     )
@@
       (project "leaf"
         (path "/e3b58043-16a3-43c8-9fad-9c9784eebfa4/cc9fb3ac-19c3-47a8-ba7d-678b4d514ff0"
-          (reference "#FLG02") (unit 1)
+          (reference "#FLG02003") (unit 1)
         )
       )
@@
   (symbol (lib_id "power:GNDA") (at 186.69 124.46 0) (unit 1)
     (in_bom yes) (on_board yes) (dnp no) (fields_autoplaced)
-    (property "Reference" "#PWR0147" (at 186.69 130.81 0)
+    (property "Reference" "#PWR02005" (at 186.69 130.81 0)
       (effects (font (size 1.27 1.27)) hide)
     )
@@
       (project "leaf"
         (path "/e3b58043-16a3-43c8-9fad-9c9784eebfa4/cc9fb3ac-19c3-47a8-ba7d-678b4d514ff0"
-          (reference "#PWR0147") (unit 1)
+          (reference "#PWR02005") (unit 1)
         )
       )
@@
         )
         (path "/e3b58043-16a3-43c8-9fad-9c9784eebfa4/cc9fb3ac-19c3-47a8-ba7d-678b4d514ff0"
-          (reference "#PWR021") (unit 1)
+          (reference "#PWR02008") (unit 1)
         )
       )
@@
   (symbol (lib_id "power:PWR_FLAG") (at 177.8 91.44 0) (unit 1)
     (in_bom yes) (on_board yes) (dnp no) (fields_autoplaced)
-    (property "Reference" "#FLG012" (at 177.8 89.535 0)
+    (property "Reference" "#FLG02001" (at 177.8 89.535 0)
       (effects (font (size 1.27 1.27)) hide)
     )
@@
       (project "leaf"
         (path "/e3b58043-16a3-43c8-9fad-9c9784eebfa4/cc9fb3ac-19c3-47a8-ba7d-678b4d514ff0"
-          (reference "#FLG012") (unit 1)
+          (reference "#FLG02001") (unit 1)
         )
       )
@@
         )
         (path "/e3b58043-16a3-43c8-9fad-9c9784eebfa4/cc9fb3ac-19c3-47a8-ba7d-678b4d514ff0"
-          (reference "NT1") (unit 1)
-        )
-      )
+          (reference "NT2001") (unit 1)
+        )
+      )

Commit message: move DDR power decoupling capacitors into DDR4 Sheet
Parts:
- renumbered U2001 to U1
Changed lines of the file:
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@@
   (symbol (lib_id "Leaf_Converter_DCDC:BL8039") (at 86.36 97.79 0) (unit 1)
     (in_bom yes) (on_board yes) (dnp no) (fields_autoplaced)
-    (property "Reference" "U2001" (at 88.9 92.3671 0)
+    (property "Reference" "U1" (at 88.9 92.3671 0)
       (effects (font (size 1.27 1.27)))
     )
@@
       (project "leaf"
         (path "/e3b58043-16a3-43c8-9fad-9c9784eebfa4/cc9fb3ac-19c3-47a8-ba7d-678b4d514ff0"
-          (reference "U2001") (unit 1)
+          (reference "U1") (unit 1)
         )
       )
@@
         )
         (path "/e3b58043-16a3-43c8-9fad-9c9784eebfa4/cc9fb3ac-19c3-47a8-ba7d-678b4d514ff0"
-          (reference "#PWR02011") (unit 1)
+          (reference "#PWR011") (unit 1)
         )
       )
@@
         )
         (path "/e3b58043-16a3-43c8-9fad-9c9784eebfa4/cc9fb3ac-19c3-47a8-ba7d-678b4d514ff0"
-          (reference "#PWR02010") (unit 1)
+          (reference "#PWR010") (unit 1)
         )
       )
@@
         )
         (path "/e3b58043-16a3-43c8-9fad-9c9784eebfa4/cc9fb3ac-19c3-47a8-ba7d-678b4d514ff0"
-          (reference "C2002") (unit 1)
+          (reference "C2") (unit 1)
         )
       )
@@
   (symbol (lib_id "power:GND") (at 200.66 49.53 0) (unit 1)
     (in_bom yes) (on_board yes) (dnp no) (fields_autoplaced)
-    (property "Reference" "#PWR02006" (at 200.66 55.88 0)
+    (property "Reference" "#PWR06" (at 200.66 55.88 0)
       (effects (font (size 1.27 1.27)) hide)
     )
@@
       (project "leaf"
         (path "/e3b58043-16a3-43c8-9fad-9c9784eebfa4/cc9fb3ac-19c3-47a8-ba7d-678b4d514ff0"
-          (reference "#PWR02006") (unit 1)
+          (reference "#PWR06") (unit 1)
         )
       )
@@
         )
         (path "/e3b58043-16a3-43c8-9fad-9c9784eebfa4/cc9fb3ac-19c3-47a8-ba7d-678b4d514ff0"
-          (reference "C2004") (unit 1)
+          (reference "C4") (unit 1)
         )
       )
@@
         )
         (path "/e3b58043-16a3-43c8-9fad-9c9784eebfa4/cc9fb3ac-19c3-47a8-ba7d-678b4d514ff0"
-          (reference "R2002") (unit 1)
+          (reference "R2") (unit 1)
         )
       )
@@
         )
         (path "/e3b58043-16a3-43c8-9fad-9c9784eebfa4/cc9fb3ac-19c3-47a8-ba7d-678b4d514ff0"
-          (reference "C2003") (unit 1)
+          (reference "C3") (unit 1)
         )
       )
@@
   (symbol (lib_id "power:GNDA") (at 74.93 124.46 0) (unit 1)
     (in_bom yes) (on_board yes) (dnp no) (fields_autoplaced)
-    (property "Reference" "#PWR02002" (at 74.93 130.81 0)
+    (property "Reference" "#PWR02" (at 74.93 130.81 0)
       (effects (font (size 1.27 1.27)) hide)
     )
@@
       (project "leaf"
         (path "/e3b58043-16a3-43c8-9fad-9c9784eebfa4/cc9fb3ac-19c3-47a8-ba7d-678b4d514ff0"
-          (reference "#PWR02002") (unit 1)
+          (reference "#PWR02") (unit 1)
         )
       )
@@
         )
         (path "/e3b58043-16a3-43c8-9fad-9c9784eebfa4/cc9fb3ac-19c3-47a8-ba7d-678b4d514ff0"
-          (reference "L2001") (unit 1)
+          (reference "L1") (unit 1)
         )
       )
@@
   (symbol (lib_id "power:PWR_FLAG") (at 234.95 43.18 0) (unit 1)
     (in_bom yes) (on_board yes) (dnp no) (fields_autoplaced)
-    (property "Reference" "#FLG02005" (at 234.95 41.275 0)
+    (property "Reference" "#FLG05" (at 234.95 41.275 0)
       (effects (font (size 1.27 1.27)) hide)
     )
@@
       (project "leaf"
         (path "/e3b58043-16a3-43c8-9fad-9c9784eebfa4/cc9fb3ac-19c3-47a8-ba7d-678b4d514ff0"
-          (reference "#FLG02005") (unit 1)
+          (reference "#FLG05") (unit 1)
         )
       )
@@
         )
         (path "/e3b58043-16a3-43c8-9fad-9c9784eebfa4/cc9fb3ac-19c3-47a8-ba7d-678b4d514ff0"
-          (reference "C2005") (unit 1)
+          (reference "C5") (unit 1)
         )
       )
@@
   (symbol (lib_id "power:GNDA") (at 43.18 111.76 0) (unit 1)
     (in_bom yes) (on_board yes) (dnp no) (fields_autoplaced)
-    (property "Reference" "#PWR02001" (at 43.18 118.11 0)
+    (property "Reference" "#PWR01" (at 43.18 118.11 0)
       (effects (font (size 1.27 1.27)) hide)
     )
@@
       (project "leaf"
         (path "/e3b58043-16a3-43c8-9fad-9c9784eebfa4/cc9fb3ac-19c3-47a8-ba7d-678b4d514ff0"
-          (reference "#PWR02001") (unit 1)
+          (reference "#PWR01") (unit 1)
         )
       )
@@
         )
         (path "/e3b58043-16a3-43c8-9fad-9c9784eebfa4/cc9fb3ac-19c3-47a8-ba7d-678b4d514ff0"
-          (reference "#PWR02007") (unit 1)
+          (reference "#PWR07") (unit 1)
         )
       )
@@
         )
         (path "/e3b58043-16a3-43c8-9fad-9c9784eebfa4/cc9fb3ac-19c3-47a8-ba7d-678b4d514ff0"
-          (reference "R2003") (unit 1)
+          (reference "R3") (unit 1)
         )
       )
@@
   (symbol (lib_id "power:GNDA") (at 88.9 124.46 0) (unit 1)
     (in_bom yes) (on_board yes) (dnp no) (fields_autoplaced)
-    (property "Reference" "#PWR02003" (at 88.9 130.81 0)
+    (property "Reference" "#PWR03" (at 88.9 130.81 0)
       (effects (font (size 1.27 1.27)) hide)
     )
@@
       (project "leaf"
         (path "/e3b58043-16a3-43c8-9fad-9c9784eebfa4/cc9fb3ac-19c3-47a8-ba7d-678b4d514ff0"
-          (reference "#PWR02003") (unit 1)
+          (reference "#PWR03") (unit 1)
         )
       )
@@
         )
         (path "/e3b58043-16a3-43c8-9fad-9c9784eebfa4/cc9fb3ac-19c3-47a8-ba7d-678b4d514ff0"
-          (reference "C2006") (unit 1)
+          (reference "C6") (unit 1)
         )
       )
@@
   (symbol (lib_id "power:PWR_FLAG") (at 185.42 44.45 0) (unit 1)
     (in_bom yes) (on_board yes) (dnp no) (fields_autoplaced)
-    (property "Reference" "#FLG02002" (at 185.42 42.545 0)
+    (property "Reference" "#FLG02" (at 185.42 42.545 0)
       (effects (font (size 1.27 1.27)) hide)
     )
@@
       (project "leaf"
         (path "/e3b58043-16a3-43c8-9fad-9c9784eebfa4/cc9fb3ac-19c3-47a8-ba7d-678b4d514ff0"
-          (reference "#FLG02002") (unit 1)
+          (reference "#FLG02") (unit 1)
         )
       )
@@
         )
         (path "/e3b58043-16a3-43c8-9fad-9c9784eebfa4/cc9fb3ac-19c3-47a8-ba7d-678b4d514ff0"
-          (reference "C2001") (unit 1)
+          (reference "C1") (unit 1)
         )
       )
@@
         )
         (path "/e3b58043-16a3-43c8-9fad-9c9784eebfa4/cc9fb3ac-19c3-47a8-ba7d-678b4d514ff0"
-          (reference "#PWR02009") (unit 1)
+          (reference "#PWR09") (unit 1)
         )
       )
@@
         )
         (path "/e3b58043-16a3-43c8-9fad-9c9784eebfa4/cc9fb3ac-19c3-47a8-ba7d-678b4d514ff0"
-          (reference "R2001") (unit 1)
+          (reference "R1") (unit 1)
         )
       )
@@
   (symbol (lib_id "power:GNDA") (at 166.37 154.94 90) (unit 1)
     (in_bom yes) (on_board yes) (dnp no) (fields_autoplaced)
-    (property "Reference" "#PWR02004" (at 172.72 154.94 0)
+    (property "Reference" "#PWR04" (at 172.72 154.94 0)
       (effects (font (size 1.27 1.27)) hide)
     )
@@
       (project "leaf"
         (path "/e3b58043-16a3-43c8-9fad-9c9784eebfa4/cc9fb3ac-19c3-47a8-ba7d-678b4d514ff0"
-          (reference "#PWR02004") (unit 1)
+          (reference "#PWR04") (unit 1)
         )
       )
@@
         )
         (path "/e3b58043-16a3-43c8-9fad-9c9784eebfa4/cc9fb3ac-19c3-47a8-ba7d-678b4d514ff0"
-          (reference "R2004") (unit 1)
+          (reference "R4") (unit 1)
         )
       )
@@
   (symbol (lib_id "power:PWR_FLAG") (at 220.98 43.18 0) (unit 1)
     (in_bom yes) (on_board yes) (dnp no) (fields_autoplaced)
-    (property "Reference" "#FLG02004" (at 220.98 41.275 0)
+    (property "Reference" "#FLG04" (at 220.98 41.275 0)
       (effects (font (size 1.27 1.27)) hide)
     )
@@
       (project "leaf"
         (path "/e3b58043-16a3-43c8-9fad-9c9784eebfa4/cc9fb3ac-19c3-47a8-ba7d-678b4d514ff0"
-          (reference "#FLG02004") (unit 1)
+          (reference "#FLG04") (unit 1)
         )
       )
@@
   (symbol (lib_id "power:PWR_FLAG") (at 205.74 43.18 0) (unit 1)
     (in_bom yes) (on_board yes) (dnp no) (fields_autoplaced)
-    (property "Reference" "#FLG02003" (at 205.74 41.275 0)
+    (property "Reference" "#FLG03" (at 205.74 41.275 0)
       (effects (font (size 1.27 1.27)) hide)
     )
@@
       (project "leaf"
         (path "/e3b58043-16a3-43c8-9fad-9c9784eebfa4/cc9fb3ac-19c3-47a8-ba7d-678b4d514ff0"
-          (reference "#FLG02003") (unit 1)
+          (reference "#FLG03") (unit 1)
         )
       )
@@
   (symbol (lib_id "power:GNDA") (at 186.69 124.46 0) (unit 1)
     (in_bom yes) (on_board yes) (dnp no) (fields_autoplaced)
-    (property "Reference" "#PWR02005" (at 186.69 130.81 0)
+    (property "Reference" "#PWR05" (at 186.69 130.81 0)
       (effects (font (size 1.27 1.27)) hide)
     )
@@
       (project "leaf"
         (path "/e3b58043-16a3-43c8-9fad-9c9784eebfa4/cc9fb3ac-19c3-47a8-ba7d-678b4d514ff0"
-          (reference "#PWR02005") (unit 1)
+          (reference "#PWR05") (unit 1)
         )
       )
@@
         )
         (path "/e3b58043-16a3-43c8-9fad-9c9784eebfa4/cc9fb3ac-19c3-47a8-ba7d-678b4d514ff0"
-          (reference "#PWR02008") (unit 1)
+          (reference "#PWR08") (unit 1)
         )
       )
@@
   (symbol (lib_id "power:PWR_FLAG") (at 177.8 91.44 0) (unit 1)
     (in_bom yes) (on_board yes) (dnp no) (fields_autoplaced)
-    (property "Reference" "#FLG02001" (at 177.8 89.535 0)
+    (property "Reference" "#FLG01" (at 177.8 89.535 0)
       (effects (font (size 1.27 1.27)) hide)
     )
@@
       (project "leaf"
         (path "/e3b58043-16a3-43c8-9fad-9c9784eebfa4/cc9fb3ac-19c3-47a8-ba7d-678b4d514ff0"
-          (reference "#FLG02001") (unit 1)
+          (reference "#FLG01") (unit 1)
         )
       )
@@
         )
         (path "/e3b58043-16a3-43c8-9fad-9c9784eebfa4/cc9fb3ac-19c3-47a8-ba7d-678b4d514ff0"
-          (reference "NT2001") (unit 1)
-        )
-      )
+          (reference "NT1") (unit 1)
+        )
+      )

Commit message: added README and license
Other:
- company: Qingdao IotPi Information Technology -> Yang Hongbo
- title: Leaf RV1126 Power -> Leaf RV1126
Changed lines of the file:
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@@
   (paper "A4")
   (title_block
-    (title "Leaf RV1126 Power")
-    (date "2023-02-25")
+    (title "Leaf RV1126")
+    (date "2023-06-07")
     (rev "1")
-    (company "Qingdao IotPi Information Technology")
+    (company "Yang Hongbo")
+    (comment 1 "License: CC BY-SA")
   )
   (junction (at 124.46 154.94) (diameter 0) (color 0 0 0 0)

Commit message: replaced Leaf specified symbols with unified iotpi symbols
Parts:
- U1: symbol Leaf_Converter_DCDC:BL8039 -> IotPi_Converter_DCDC:BL8039
Changed lines of the file:
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@@
     (effects (font (size 1.27 1.27)) (justify right))
   )
-  (symbol (lib_id "Leaf_Converter_DCDC:BL8039") (at 86.36 97.79 0) (unit 1)
+  (symbol (lib_id "IotPi_Converter_DCDC:BL8039") (at 86.36 97.79 0) (unit 1)
     (in_bom yes) (on_board yes) (dnp no) (fields_autoplaced)
     (property "Reference" "U1" (at 88.9 92.3671 0)
@@
       (effects (font (size 1.27 1.27)) hide)
     )
+    (property "Description" "" (at 86.36 97.79 0)
+      (effects (font (size 1.27 1.27)) hide)
+    )
