File: VCCIO4.kicad_sch (KiCad schematic)
At the start: 14 parts, among them J7001 MIPI-CSI, U3001 rv1126/rv1109

Commit message: move DDR power decoupling capacitors into DDR4 Sheet
Parts:
- renumbered J7001 to J2, U3001 to U2
Changed lines of the file:
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@@
         )
         (path "/e3b58043-16a3-43c8-9fad-9c9784eebfa4/bca9f05a-f031-46a4-95a9-25be55b42bf6"
-          (reference "#PWR07011") (unit 1)
+          (reference "#PWR037") (unit 1)
         )
       )
@@
         )
         (path "/e3b58043-16a3-43c8-9fad-9c9784eebfa4/bca9f05a-f031-46a4-95a9-25be55b42bf6"
-          (reference "C7008") (unit 1)
+          (reference "C31") (unit 1)
         )
       )
@@
         )
         (path "/e3b58043-16a3-43c8-9fad-9c9784eebfa4/bca9f05a-f031-46a4-95a9-25be55b42bf6"
-          (reference "R7004") (unit 1)
+          (reference "R23") (unit 1)
         )
       )
@@
   (symbol (lib_id "Connector_Generic_MountingPin:Conn_01x24_MountingPin") (at 275.59 68.58 0) (unit 1)
     (in_bom yes) (on_board yes) (dnp no)
-    (property "Reference" "J7001" (at 276.225 37.5539 0)
+    (property "Reference" "J2" (at 276.225 37.5539 0)
       (effects (font (size 1.27 1.27)))
     )
@@
       (project "leaf"
         (path "/e3b58043-16a3-43c8-9fad-9c9784eebfa4/bca9f05a-f031-46a4-95a9-25be55b42bf6"
-          (reference "J7001") (unit 1)
+          (reference "J2") (unit 1)
         )
       )
@@
         )
         (path "/e3b58043-16a3-43c8-9fad-9c9784eebfa4/bca9f05a-f031-46a4-95a9-25be55b42bf6"
-          (reference "R7001") (unit 1)
+          (reference "R20") (unit 1)
         )
       )
@@
         )
         (path "/e3b58043-16a3-43c8-9fad-9c9784eebfa4/bca9f05a-f031-46a4-95a9-25be55b42bf6"
-          (reference "C7006") (unit 1)
+          (reference "C29") (unit 1)
         )
       )
@@
   (symbol (lib_id "power:PWR_FLAG") (at 114.3 171.45 0) (unit 1)
     (in_bom yes) (on_board yes) (dnp no) (fields_autoplaced)
-    (property "Reference" "#FLG07002" (at 114.3 169.545 0)
+    (property "Reference" "#FLG07" (at 114.3 169.545 0)
       (effects (font (size 1.27 1.27)) hide)
     )
@@
       (project "leaf"
         (path "/e3b58043-16a3-43c8-9fad-9c9784eebfa4/bca9f05a-f031-46a4-95a9-25be55b42bf6"
-          (reference "#FLG07002") (unit 1)
+          (reference "#FLG07") (unit 1)
         )
       )
@@
         )
         (path "/e3b58043-16a3-43c8-9fad-9c9784eebfa4/bca9f05a-f031-46a4-95a9-25be55b42bf6"
-          (reference "C7002") (unit 1)
+          (reference "C25") (unit 1)
         )
       )
@@
         )
         (path "/e3b58043-16a3-43c8-9fad-9c9784eebfa4/bca9f05a-f031-46a4-95a9-25be55b42bf6"
-          (reference "C7005") (unit 1)
+          (reference "C28") (unit 1)
         )
       )
@@
         )
         (path "/e3b58043-16a3-43c8-9fad-9c9784eebfa4/bca9f05a-f031-46a4-95a9-25be55b42bf6"
-          (reference "C7001") (unit 1)
+          (reference "C24") (unit 1)
         )
       )
@@
         )
         (path "/e3b58043-16a3-43c8-9fad-9c9784eebfa4/bca9f05a-f031-46a4-95a9-25be55b42bf6"
-          (reference "C7003") (unit 1)
+          (reference "C26") (unit 1)
         )
       )
@@
         )
         (path "/e3b58043-16a3-43c8-9fad-9c9784eebfa4/bca9f05a-f031-46a4-95a9-25be55b42bf6"
-          (reference "#PWR07009") (unit 1)
+          (reference "#PWR036") (unit 1)
         )
       )
@@
         )
         (path "/e3b58043-16a3-43c8-9fad-9c9784eebfa4/bca9f05a-f031-46a4-95a9-25be55b42bf6"
-          (reference "#PWR07004") (unit 1)
+          (reference "#PWR031") (unit 1)
         )
       )
@@
         )
         (path "/e3b58043-16a3-43c8-9fad-9c9784eebfa4/bca9f05a-f031-46a4-95a9-25be55b42bf6"
-          (reference "#PWR07010") (unit 1)
+          (reference "#PWR038") (unit 1)
         )
       )
@@
   (symbol (lib_id "power:GNDA") (at 109.22 185.42 0) (mirror y) (unit 1)
     (in_bom yes) (on_board yes) (dnp no) (fields_autoplaced)
-    (property "Reference" "#PWR07003" (at 109.22 191.77 0)
+    (property "Reference" "#PWR030" (at 109.22 191.77 0)
       (effects (font (size 1.27 1.27)) hide)
     )
@@
       (project "leaf"
         (path "/e3b58043-16a3-43c8-9fad-9c9784eebfa4/bca9f05a-f031-46a4-95a9-25be55b42bf6"
-          (reference "#PWR07003") (unit 1)
+          (reference "#PWR030") (unit 1)
         )
       )
@@
   (symbol (lib_id "power:GNDA") (at 64.77 184.15 0) (mirror y) (unit 1)
     (in_bom yes) (on_board yes) (dnp no) (fields_autoplaced)
-    (property "Reference" "#PWR07001" (at 64.77 190.5 0)
+    (property "Reference" "#PWR028" (at 64.77 190.5 0)
       (effects (font (size 1.27 1.27)) hide)
     )
@@
       (project "leaf"
         (path "/e3b58043-16a3-43c8-9fad-9c9784eebfa4/bca9f05a-f031-46a4-95a9-25be55b42bf6"
-          (reference "#PWR07001") (unit 1)
+          (reference "#PWR028") (unit 1)
         )
       )
@@
   (symbol (lib_id "power:GNDD") (at 250.19 40.64 270) (unit 1)
     (in_bom yes) (on_board yes) (dnp no) (fields_autoplaced)
-    (property "Reference" "#PWR07005" (at 243.84 40.64 0)
+    (property "Reference" "#PWR032" (at 243.84 40.64 0)
       (effects (font (size 1.27 1.27)) hide)
     )
@@
       (project "leaf"
         (path "/e3b58043-16a3-43c8-9fad-9c9784eebfa4/bca9f05a-f031-46a4-95a9-25be55b42bf6"
-          (reference "#PWR07005") (unit 1)
+          (reference "#PWR032") (unit 1)
         )
       )
@@
   (symbol (lib_id "power:GNDD") (at 250.19 88.9 270) (unit 1)
     (in_bom yes) (on_board yes) (dnp no) (fields_autoplaced)
-    (property "Reference" "#PWR07008" (at 243.84 88.9 0)
+    (property "Reference" "#PWR035" (at 243.84 88.9 0)
       (effects (font (size 1.27 1.27)) hide)
     )
@@
       (project "leaf"
         (path "/e3b58043-16a3-43c8-9fad-9c9784eebfa4/bca9f05a-f031-46a4-95a9-25be55b42bf6"
-          (reference "#PWR07008") (unit 1)
+          (reference "#PWR035") (unit 1)
         )
       )
@@
   (symbol (lib_id "power:PWR_FLAG") (at 69.85 170.18 0) (unit 1)
     (in_bom yes) (on_board yes) (dnp no) (fields_autoplaced)
-    (property "Reference" "#FLG07001" (at 69.85 168.275 0)
+    (property "Reference" "#FLG06" (at 69.85 168.275 0)
       (effects (font (size 1.27 1.27)) hide)
     )
@@
       (project "leaf"
         (path "/e3b58043-16a3-43c8-9fad-9c9784eebfa4/bca9f05a-f031-46a4-95a9-25be55b42bf6"
-          (reference "#FLG07001") (unit 1)
+          (reference "#FLG06") (unit 1)
         )
       )
@@
         )
         (path "/e3b58043-16a3-43c8-9fad-9c9784eebfa4/bca9f05a-f031-46a4-95a9-25be55b42bf6"
-          (reference "R7002") (unit 1)
+          (reference "R21") (unit 1)
         )
       )
@@
         )
         (path "/e3b58043-16a3-43c8-9fad-9c9784eebfa4/bca9f05a-f031-46a4-95a9-25be55b42bf6"
-          (reference "C7004") (unit 1)
+          (reference "C27") (unit 1)
         )
       )
@@
   (symbol (lib_id "power:GND") (at 96.52 83.82 0) (unit 1)
     (in_bom yes) (on_board yes) (dnp no) (fields_autoplaced)
-    (property "Reference" "#PWR07002" (at 96.52 90.17 0)
+    (property "Reference" "#PWR029" (at 96.52 90.17 0)
       (effects (font (size 1.27 1.27)) hide)
     )
@@
       (project "leaf"
         (path "/e3b58043-16a3-43c8-9fad-9c9784eebfa4/bca9f05a-f031-46a4-95a9-25be55b42bf6"
-          (reference "#PWR07002") (unit 1)
+          (reference "#PWR029") (unit 1)
         )
       )
@@
   (symbol (lib_id "power:GNDD") (at 250.19 81.28 270) (unit 1)
     (in_bom yes) (on_board yes) (dnp no) (fields_autoplaced)
-    (property "Reference" "#PWR07007" (at 243.84 81.28 0)
+    (property "Reference" "#PWR034" (at 243.84 81.28 0)
       (effects (font (size 1.27 1.27)) hide)
     )
@@
       (project "leaf"
         (path "/e3b58043-16a3-43c8-9fad-9c9784eebfa4/bca9f05a-f031-46a4-95a9-25be55b42bf6"
-          (reference "#PWR07007") (unit 1)
+          (reference "#PWR034") (unit 1)
         )
       )
@@
   (symbol (lib_id "power:GNDD") (at 250.19 55.88 270) (unit 1)
     (in_bom yes) (on_board yes) (dnp no) (fields_autoplaced)
-    (property "Reference" "#PWR07006" (at 243.84 55.88 0)
+    (property "Reference" "#PWR033" (at 243.84 55.88 0)
       (effects (font (size 1.27 1.27)) hide)
     )
@@
       (project "leaf"
         (path "/e3b58043-16a3-43c8-9fad-9c9784eebfa4/bca9f05a-f031-46a4-95a9-25be55b42bf6"
-          (reference "#PWR07006") (unit 1)
+          (reference "#PWR033") (unit 1)
         )
       )
@@
   (symbol (lib_id "CPU_Rockchip:rv1126_rv1109") (at 55.88 57.15 0) (unit 9)
     (in_bom yes) (on_board yes) (dnp no) (fields_autoplaced)
-    (property "Reference" "U3001" (at 55.88 30.1371 0)
+    (property "Reference" "U2" (at 55.88 30.1371 0)
       (effects (font (size 1.27 1.27)))
     )
@@
       (project "leaf"
         (path "/e3b58043-16a3-43c8-9fad-9c9784eebfa4/bca9f05a-f031-46a4-95a9-25be55b42bf6"
-          (reference "U3001") (unit 9)
+          (reference "U2") (unit 9)
         )
       )
@@
         )
         (path "/e3b58043-16a3-43c8-9fad-9c9784eebfa4/bca9f05a-f031-46a4-95a9-25be55b42bf6"
-          (reference "R7003") (unit 1)
+          (reference "R22") (unit 1)
         )
       )
@@
   (symbol (lib_id "CPU_Rockchip:rv1126_rv1109") (at 161.29 57.15 0) (unit 15)
     (in_bom yes) (on_board yes) (dnp no) (fields_autoplaced)
-    (property "Reference" "U3001" (at 161.29 22.5171 0)
+    (property "Reference" "U2" (at 161.29 22.5171 0)
       (effects (font (size 1.27 1.27)))
     )
@@
       (project "leaf"
         (path "/e3b58043-16a3-43c8-9fad-9c9784eebfa4/bca9f05a-f031-46a4-95a9-25be55b42bf6"
-          (reference "U3001") (unit 15)
+          (reference "U2") (unit 15)
         )
       )
@@
         )
         (path "/e3b58043-16a3-43c8-9fad-9c9784eebfa4/bca9f05a-f031-46a4-95a9-25be55b42bf6"
-          (reference "C7007") (unit 1)
-        )
-      )
+          (reference "C30") (unit 1)
+        )
+      )

Commit message: remove all warnings
Changed lines of the file:
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@@
     (effects (font (size 1.27 1.27)) (justify left bottom))
-  )
-  (label "DGND3" (at 259.08 58.42 180) (fields_autoplaced)
-    (effects (font (size 1.27 1.27)) (justify right bottom))
   )
   (label "MIPI_RX0_D1N" (at 200.66 41.91 0) (fields_autoplaced)
@@
   )
   (label "MIPI_CSI_PWR0" (at 241.3 45.72 180) (fields_autoplaced)
-    (effects (font (size 1.27 1.27)) (justify right bottom))
-  )
-  (label "DGND1" (at 259.08 43.18 180) (fields_autoplaced)
     (effects (font (size 1.27 1.27)) (justify right bottom))
   )
@@
   )
   (label "VCC_0V8" (at 85.09 166.37 180) (fields_autoplaced)
-    (effects (font (size 1.27 1.27)) (justify right bottom))
-  )
-  (label "DGND0" (at 259.08 40.64 180) (fields_autoplaced)
     (effects (font (size 1.27 1.27)) (justify right bottom))
   )
@@
     (effects (font (size 1.27 1.27)) (justify right bottom))
   )
-  (label "DGND2" (at 259.08 55.88 180) (fields_autoplaced)
-    (effects (font (size 1.27 1.27)) (justify right bottom))
-  )
   (label "MIPI_CSI_PWR0" (at 104.14 63.5 0) (fields_autoplaced)
     (effects (font (size 1.27 1.27)) (justify left bottom))
@@
     (effects (font (size 1.27 1.27)) (justify right bottom))
   )
-  (label "DGND4" (at 259.08 81.28 180) (fields_autoplaced)
-    (effects (font (size 1.27 1.27)) (justify right bottom))
-  )
   (label "MIPI_CSI_I2C_SDA" (at 104.14 43.18 0) (fields_autoplaced)
     (effects (font (size 1.27 1.27)) (justify left bottom))
@@
     (effects (font (size 1.27 1.27)) (justify left bottom))
   )
-  (label "DGND5" (at 259.08 88.9 180) (fields_autoplaced)
-    (effects (font (size 1.27 1.27)) (justify right bottom))
-  )
   (label "MIPI_RX0_D3P" (at 241.3 78.74 180) (fields_autoplaced)

Commit message: added README and license
Other:
- company: Qingdao IotPi Information Technology -> Yang Hongbo
- title: Leaf RV1126 RK809 Camera -> Leaf RV1126
Changed lines of the file:
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@@
   (paper "A4")
   (title_block
-    (title "Leaf RV1126 RK809 Camera")
-    (date "2023-02-25")
+    (title "Leaf RV1126")
+    (date "2023-06-07")
     (rev "1")
-    (company "Qingdao IotPi Information Technology")
+    (company "Yang Hongbo")
+    (comment 1 "License: CC BY-SA")
   )
   (junction (at 41.91 105.41) (diameter 0) (color 0 0 0 0)

Commit message: replaced Leaf specified symbols with unified iotpi symbols
Parts:
- U2: symbol CPU_Rockchip:rv1126_rv1109 -> IotPi_CPU_Rockchip:rv1126_rv1109
Changed lines of the file:
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@@
     )
   )
-  (symbol (lib_id "CPU_Rockchip:rv1126_rv1109") (at 55.88 57.15 0) (unit 9)
+  (symbol (lib_id "IotPi_CPU_Rockchip:rv1126_rv1109") (at 55.88 57.15 0) (unit 9)
     (in_bom yes) (on_board yes) (dnp no) (fields_autoplaced)
     (property "Reference" "U2" (at 55.88 30.1371 0)
@@
       (effects (font (size 1.27 1.27)))
     )
-    (property "Footprint" "Rockchip_SoC:Rockchip_RV1126_FCCSP409LD_14.0x14.0mm" (at 87.63 83.82 0)
-      (effects (font (size 1.27 1.27)) hide)
-    )
-    (property "Datasheet" "" (at 87.63 83.82 0)
+    (property "Footprint" "Rockchip_SoC:Rockchip_RV1126_FCCSP409LD_14.0x14.0mm" (at 87.63 104.14 0)
+      (effects (font (size 1.27 1.27)) hide)
+    )
+    (property "Datasheet" "" (at 87.63 104.14 0)
       (effects (font (size 1.27 1.27)) hide)
     )
@@
     )
   )
-  (symbol (lib_id "CPU_Rockchip:rv1126_rv1109") (at 161.29 57.15 0) (unit 15)
+  (symbol (lib_id "IotPi_CPU_Rockchip:rv1126_rv1109") (at 161.29 57.15 0) (unit 15)
     (in_bom yes) (on_board yes) (dnp no) (fields_autoplaced)
     (property "Reference" "U2" (at 161.29 22.5171 0)
@@
       (effects (font (size 1.27 1.27)))
     )
-    (property "Footprint" "Rockchip_SoC:Rockchip_RV1126_FCCSP409LD_14.0x14.0mm" (at 193.04 83.82 0)
-      (effects (font (size 1.27 1.27)) hide)
-    )
-    (property "Datasheet" "" (at 193.04 83.82 0)
-      (effects (font (size 1.27 1.27)) hide)
-    )
+    (property "Footprint" "Rockchip_SoC:Rockchip_RV1126_FCCSP409LD_14.0x14.0mm" (at 193.04 104.14 0)
+      (effects (font (size 1.27 1.27)) hide)
+    )
+    (property "Datasheet" "" (at 193.04 104.14 0)
+      (effects (font (size 1.27 1.27)) hide)
+    )
