File: VCCIO4.kicad_sch (KiCad schematic)
At the start: 14 parts, among them J2 MIPI-CSI, U2 rv1126/rv1109

Commit message: replaced Leaf libraries with combined libraries
Parts:
- U2: footprint Rockchip_SoC:Rockchip_RV1126_FCCSP409LD_14.0x14.0mm -> IotPi_Rockchip_SoC:Rockchip_RV1126_FCCSP409LD_14.0x14.0mm
Changed lines of the file:
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@@
       (effects (font (size 1.27 1.27)))
     )
-    (property "Footprint" "Rockchip_SoC:Rockchip_RV1126_FCCSP409LD_14.0x14.0mm" (at 87.63 104.14 0)
+    (property "Footprint" "IotPi_Rockchip_SoC:Rockchip_RV1126_FCCSP409LD_14.0x14.0mm" (at 87.63 104.14 0)
       (effects (font (size 1.27 1.27)) hide)
     )
@@
       (effects (font (size 1.27 1.27)))
     )
-    (property "Footprint" "Rockchip_SoC:Rockchip_RV1126_FCCSP409LD_14.0x14.0mm" (at 193.04 104.14 0)
-      (effects (font (size 1.27 1.27)) hide)
-    )
+    (property "Footprint" "IotPi_Rockchip_SoC:Rockchip_RV1126_FCCSP409LD_14.0x14.0mm" (at 193.04 104.14 0)
+      (effects (font (size 1.27 1.27)) hide)
+    )
