File: SoC_OSC_PLL.kicad_sch (KiCad schematic)
At the start: 10 parts, among them U1 rv1126/rv1109, Y3 24MHz ±10ppm 10pF

Commit message: replaced Leaf specified symbols with unified iotpi symbols
Parts:
- U1: symbol CPU_Rockchip:rv1126_rv1109 -> IotPi_CPU_Rockchip:rv1126_rv1109
Changed lines of the file:
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@@
     )
   )
-  (symbol (lib_id "CPU_Rockchip:rv1126_rv1109") (at 48.26 109.22 0) (unit 3)
+  (symbol (lib_id "IotPi_CPU_Rockchip:rv1126_rv1109") (at 48.26 109.22 0) (unit 3)
     (in_bom yes) (on_board yes) (dnp no) (fields_autoplaced)
     (property "Reference" "U1" (at 48.26 77.1271 0)
@@
       (effects (font (size 1.27 1.27)))
     )
-    (property "Footprint" "Rockchip_SoC:Rockchip_RV1126_FCCSP409LD_14.0x14.0mm" (at 80.01 135.89 0)
+    (property "Footprint" "Rockchip_SoC:Rockchip_RV1126_FCCSP409LD_14.0x14.0mm" (at 80.01 156.21 0)
       (effects (font (size 1.27 1.27)) hide)
     )
-    (property "Datasheet" "" (at 80.01 135.89 0)
+    (property "Datasheet" "" (at 80.01 156.21 0)
       (effects (font (size 1.27 1.27)) hide)
     )

Commit message: replaced Leaf libraries with combined libraries
Parts:
- U1: footprint Rockchip_SoC:Rockchip_RV1126_FCCSP409LD_14.0x14.0mm -> IotPi_Rockchip_SoC:Rockchip_RV1126_FCCSP409LD_14.0x14.0mm
Changed lines of the file:
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@@
       (effects (font (size 1.27 1.27)))
     )
-    (property "Footprint" "Rockchip_SoC:Rockchip_RV1126_FCCSP409LD_14.0x14.0mm" (at 80.01 156.21 0)
+    (property "Footprint" "IotPi_Rockchip_SoC:Rockchip_RV1126_FCCSP409LD_14.0x14.0mm" (at 80.01 156.21 0)
       (effects (font (size 1.27 1.27)) hide)
     )
