File: VCCIO1.kicad_sch (KiCad schematic)
At the start: 19 parts, among them U2 rv1126/rv1109, U3 MTFC4GACAJCN

Commit message: replaced Leaf libraries with combined libraries
Parts:
- U2: footprint Rockchip_SoC:Rockchip_RV1126_FCCSP409LD_14.0x14.0mm -> IotPi_Rockchip_SoC:Rockchip_RV1126_FCCSP409LD_14.0x14.0mm
- U3: footprint Memory_micron:Micron_eMMC_FBGA-153_11.5x13.0mm -> IotPi_Memory_Micron:Micron_eMMC_FBGA-153_11.5x13.0mm
Changed lines of the file:
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@@
       (effects (font (size 1.27 1.27)) (justify left))
     )
-    (property "Footprint" "Memory_micron:Micron_eMMC_FBGA-153_11.5x13.0mm" (at 29.21 166.37 0)
+    (property "Footprint" "IotPi_Memory_Micron:Micron_eMMC_FBGA-153_11.5x13.0mm" (at 29.21 166.37 0)
       (effects (font (size 1.27 1.27)) hide)
     )
@@
       (effects (font (size 1.27 1.27)))
     )
-    (property "Footprint" "Memory_micron:Micron_eMMC_FBGA-153_11.5x13.0mm" (at 179.07 48.26 0)
+    (property "Footprint" "IotPi_Memory_Micron:Micron_eMMC_FBGA-153_11.5x13.0mm" (at 179.07 48.26 0)
       (effects (font (size 1.27 1.27)) hide)
     )
@@
       (effects (font (size 1.27 1.27)))
     )
-    (property "Footprint" "Rockchip_SoC:Rockchip_RV1126_FCCSP409LD_14.0x14.0mm" (at 100.33 106.68 0)
-      (effects (font (size 1.27 1.27)) hide)
-    )
+    (property "Footprint" "IotPi_Rockchip_SoC:Rockchip_RV1126_FCCSP409LD_14.0x14.0mm" (at 100.33 106.68 0)
+      (effects (font (size 1.27 1.27)) hide)
+    )
