File: VCCIO2.kicad_sch (KiCad schematic)
At the start: 19 parts, among them J1 Micro_SD_Card_Det1, U2 rv1126/rv1109

Commit message: replaced Leaf libraries with combined libraries
Parts:
- J1: footprint Leaf_Connector:microSD -> IotPi_Connector:microSD
- U2: footprint Rockchip_SoC:Rockchip_RV1126_FCCSP409LD_14.0x14.0mm -> IotPi_Rockchip_SoC:Rockchip_RV1126_FCCSP409LD_14.0x14.0mm
Changed lines of the file:
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@@
       (effects (font (size 1.27 1.27)))
     )
-    (property "Footprint" "Leaf_Connector:microSD" (at 0 99.06 0)
+    (property "Footprint" "IotPi_Connector:microSD" (at 0 99.06 0)
       (effects (font (size 1.27 1.27)) hide)
     )
@@
       (effects (font (size 1.27 1.27)))
     )
-    (property "Footprint" "Rockchip_SoC:Rockchip_RV1126_FCCSP409LD_14.0x14.0mm" (at 158.75 106.68 0)
+    (property "Footprint" "IotPi_Rockchip_SoC:Rockchip_RV1126_FCCSP409LD_14.0x14.0mm" (at 158.75 106.68 0)
       (effects (font (size 1.27 1.27)) hide)
     )
