File: WiFi.kicad_sch (KiCad schematic)
At the start: 4 parts, among them U4 AP6526, Y1 Crystal

Commit message: replaced Leaf libraries with combined libraries
Parts:
- U4: footprint Leaf_RF_Module:QFN-44_12x12_Pitch0.9mm -> IotPi_RF_Module:QFN-44_12x12_Pitch0.9mm; symbol Leaf_RF_Wifi:AP6256 -> IotPi_RF_Wifi:AP6256; now in the parts list
Changed lines of the file:
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@@
     )
   )
-  (symbol (lib_id "Leaf_RF_Wifi:AP6256") (at 148.59 73.66 0) (unit 1)
-    (in_bom no) (on_board no) (dnp yes) (fields_autoplaced)
+  (symbol (lib_id "IotPi_RF_Wifi:AP6256") (at 148.59 73.66 0) (unit 1)
+    (in_bom yes) (on_board yes) (dnp yes) (fields_autoplaced)
     (property "Reference" "U4" (at 147.955 46.6471 0)
       (effects (font (size 1.27 1.27)))
@@
       (effects (font (size 1.27 1.27)))
     )
-    (property "Footprint" "Leaf_RF_Module:QFN-44_12x12_Pitch0.9mm" (at 147.955 59.69 0)
+    (property "Footprint" "IotPi_RF_Module:QFN-44_12x12_Pitch0.9mm" (at 149.225 50.8 0)
       (effects (font (size 1.27 1.27)) hide)
     )
-    (property "Datasheet" "" (at 147.955 59.69 0)
+    (property "Datasheet" "" (at 149.225 50.8 0)
       (effects (font (size 1.27 1.27)) hide)
     )
+    (property "LCSC" "" (at 148.59 73.66 0)
+      (effects (font (size 1.27 1.27)) hide)
+    )
+    (property "Description" "" (at 148.59 73.66 0)
+      (effects (font (size 1.27 1.27)) hide)
+    )
+    (property "Vendor" "" (at 148.59 73.66 0)
+      (effects (font (size 1.27 1.27)) hide)
+    )
